Commit message: fixed wheels not loaded properly from gazebo to rviz

File: description/gazebo_control.xacro (robot description, xacro)
@@ -20,3 +20,16 @@
         </plugin>
     </gazebo>
+    <!-- Gazebo requires the use of plugins to interact with other systems such as ROS. -->
+    <!-- This plugin will publish the joint_states for the selected joints
+            (which robot_state_publisher can then use to broadcast the approprate tf). -->
+    <gazebo>
+        <plugin name="gazebo_ros_joint_state_publisher"
+            filename="libgazebo_ros_joint_state_publisher.so">
+            <update_rate>20</update_rate>
+            <joint_name>left_back_wheel-base</joint_name>
+            <joint_name>right_back_wheel-base</joint_name>
+            <joint_name>left_front_wheel-base</joint_name>
+            <joint_name>right_front_wheel-base</joint_name>
+        </plugin>
+    </gazebo>
 </robot>

File: description/robot_core.xacro (robot description, xacro)
@@ -139,5 +139,5 @@
         <axis xyz="0 0 -1"/>
     </joint>
-    <joint name="left_front_wheel-base" type="fixed">
+    <joint name="left_front_wheel-base" type="continuous">
         <parent link="base"/>
         <child link="left_front_wheel"/>
@@ -145,5 +145,5 @@
         <axis xyz="0 0 1"/>
     </joint>
-    <joint name="right_front_wheel-base" type="fixed">
+    <joint name="right_front_wheel-base" type="continuous">
         <parent link="base"/>
         <child link="right_front_wheel"/>
@@ -163,11 +163,11 @@
      <gazebo reference="left_front_wheel">
         <material>Gazebo/Blue</material>
-        <mu1 value="0.001"/>
-        <mu2 value="0.001"/>
+        <mu1 value="0.1"/>
+        <mu2 value="0.1"/>
      </gazebo>
      <gazebo reference="right_front_wheel">
         <material>Gazebo/Blue</material>
-        <mu1 value="0.001"/>
-        <mu2 value="0.001"/>
+        <mu1 value="0.1"/>
+        <mu2 value="0.1"/>
      </gazebo>
 </robot>
