Commit message: removed initial content

File: description/robot_urdf.xacro (robot description, xacro)
@@ -3,5 +3,3 @@
 <robot xmlns:xacro="http://www.ros.org/wiki/xacro"  name="robot">
     <xacro:include filename="robot_core.xacro" />
-    <!-- Example link -->
-    <link name="base_link"></link>
 </robot>

Commit message: swap between ros2 and gazebo

File: description/robot_urdf.xacro (robot description, xacro)
@@ -2,7 +2,12 @@
 <!-- loaded urdf file for robot-->
 <robot xmlns:xacro="http://www.ros.org/wiki/xacro"  name="robot">
+    <xacro:property name="use_ros2_control" value="true"/>
+    <xacro:if value="${use_ros2_control}">
+        <xacro:include filename="ros2_control.xacro"/>
+    </xacro:if>
+    <xacro:unless value="${use_ros2_control}">
+        <xacro:include filename="gazebo_control.xacro"/>
+    </xacro:unless>
     <xacro:include filename="robot_core.xacro"/>
-    <!-- <xacro:include filename="gazebo_control.xacro"/> -->
-    <xacro:include filename="ros2_control.xacro"/>
     <xacro:include filename="lidar.xacro"/>
 </robot>
