Commit message: fixed robot urdf

File: description/ros2_control.xacro (robot description, xacro)
@@ -1,5 +1,5 @@
 <?xml version="1.0"?>
 <robot xmlns:xacro="http://www.ros.org/wiki/xacro">
-    <ros2_control name="GazeboSystem" type="system">
+    <ros2_control name="botSys" type="system">
         <hardware>
             <plugin>gazebo_ros2_control/GazeboSystem</plugin>
@@ -21,11 +21,27 @@
             <state_interface name="position"/>
         </joint>
+        <joint name="left_front_wheel-base">
+            <command_interface name="velocity">
+                <param name="min">-10</param>
+                <param name="max">10</param>
+            </command_interface>
+            <state_interface name="velocity"/>
+            <state_interface name="position"/>
+        </joint>
+        <joint name="right_front_wheel-base">
+            <command_interface name="velocity">
+                <param name="min">-10</param>
+                <param name="max">10</param>
+            </command_interface>
+            <state_interface name="velocity"/>
+            <state_interface name="position"/>
+        </joint>
     </ros2_control>
     <gazebo>
-        <plugin name="gazebo_ros2_control" filename="libgazebo_ros2_control.so">
+        <plugin name="controlPlugin" filename="libgazebo_ros2_control.so">
             <parameters>$(find bot)/config/my_controllers.yaml</parameters>
         </plugin>
     </gazebo>
-    <gazebo>
+    <!-- <gazebo>
         <plugin name="gazebo_ros_joint_state_publisher"
             filename="libgazebo_ros_joint_state_publisher.so">
@@ -36,4 +52,4 @@
             <joint_name>right_front_wheel-base</joint_name>
         </plugin>
-    </gazebo>
+    </gazebo> -->
 </robot>
