Commit message: create robot  urdf

File: description/robot_core.xacro (robot description, xacro)
@@ -1,3 +1,153 @@
 <?xml version="1.0"?>
+<!-- ROBOT CORE COMPONENTS-->
+<!-- call xacro-->
 <robot xmlns:xacro="http://www.ros.org/wiki/xacro">
+    <!-- Inertial xacro-->
+    <xacro:include filename="inertial_macros.xacro"/>
+    <!-- Static Variables -->
+    <xacro:property name="left_roll" value="${-pi/2}"/>
+    <xacro:property name="right_roll" value="${pi/2}"/>
+    <!-- Independent Variables -->
+    <xacro:property name="chassis_base" value="0.3"/>
+    <xacro:property name="chassis_height" value="0.15"/>
+    <xacro:property name="chassis_mass" value="0.36"/>
+    <xacro:property name="wheel_radius" value="0.05"/>
+    <xacro:property name="wheel_length" value="0.05"/>
+    <xacro:property name="wheel_mass" value="0.1"/>
+    <!-- Dependent Variables-->
+    <xacro:property name="chassis_joint_offset" value="${-chassis_base/3}"/>
+    <xacro:property name="chassis_link_offset" value="${chassis_base/2}"/>
+    <xacro:property name="chassis_height_offset" value="${chassis_height/2}"/>
+    <xacro:property name="frontwheel_offset" value="${(chassis_base * 0.5/5) - (chassis_joint_offset)}"/>
+    <xacro:property name="backwheel_offset" value="${-(chassis_base * 0.5/5)}"/>
+    <xacro:property name="leftwheel_offset" value="${(chassis_base/2) + (wheel_length/2)}"/>
+    <xacro:property name="rightwheel_offset" value="-${(chassis_base/2) + (wheel_length/2)}"/>
+    <!-- Materials -->
+    <material name="white">
+        <color rgba="1 1 1 1" />
+    </material>
+    <material name="orange">
+        <color rgba="1 0.3 1 1" />
+    </material>
+    <material name="blue">
+        <color rgba="0.2 0.2 1 1"/>
+    </material>
+    <material name="black">
+        <color rgba="0 0 0 1"/>
+    </material>
+    <!-- links -->
+    <link name="base">
+    </link>
+    <link name="chassis">
+        <visual>
+            <origin xyz="${chassis_link_offset} 0 ${chassis_height_offset}"/>
+            <geometry>
+                <box size="${chassis_base} ${chassis_base} ${chassis_height}"/>
+            </geometry>
+            <material name="white"/>
+        </visual>
+        <collision>
+            <origin xyz="${chassis_link_offset} 0 ${chassis_height_offset}"/>
+            <geometry>
+                <box size="${chassis_base} ${chassis_base} ${chassis_height}"/>
+            </geometry>
+        </collision>
+        <xacro:inertial_box mass="${chassis_mass}" x="${chassis_base}" y="${chassis_base}" z="${chassis_height}">
+            <origin xyz="${chassis_link_offset} 0 ${chassis_height_offset}" rpy="0 0 0"/>
+        </xacro:inertial_box>
+    </link>
+    <link name="left_back_wheel">
+        <visual>
+            <geometry>
+                <cylinder radius="${wheel_radius}" length="${wheel_length}"/>
+            </geometry>
+            <material name="blue"/>
+        </visual>
+        <collision>
+            <geometry>
+                <cylinder radius="${wheel_radius}" length="${wheel_length}"/>
+            </geometry>
+        </collision>
+        <xacro:inertial_cylinder mass="${wheel_mass}" length="${wheel_length}" radius="${wheel_radius}">
+            <origin xyz="0 0 0" rpy="0 0 0"/>
+        </xacro:inertial_cylinder>
+    </link>
+    <link name="right_back_wheel">
+        <visual>
+            <geometry>
+                <cylinder radius="${wheel_radius}" length="${wheel_length}"/>
+            </geometry>
+            <material name="blue"/>
+        </visual>
+        <collision>
+            <geometry>
+                <cylinder radius="${wheel_radius}" length="${wheel_length}"/>
+            </geometry>
+        </collision>
+        <xacro:inertial_cylinder mass="${wheel_mass}" length="${wheel_length}" radius="${wheel_radius}">
+            <origin xyz="0 0 0" rpy="0 0 0"/>
+        </xacro:inertial_cylinder>
+    </link>
+    <link name="left_front_wheel">
+        <visual>
+            <geometry>
+                <cylinder radius="${wheel_radius}" length="${wheel_length}"/>
+            </geometry>
+            <material name="blue"/>
+        </visual>
+        <collision>
+            <geometry>
+                <cylinder radius="${wheel_radius}" length="${wheel_length}"/>
+            </geometry>
+        </collision>
+        <xacro:inertial_cylinder mass="${wheel_mass}" length="${wheel_length}" radius="${wheel_radius}">
+            <origin xyz="0 0 0" rpy="0 0 0"/>
+        </xacro:inertial_cylinder>
+    </link>
+    <link name="right_front_wheel">
+        <visual>
+            <geometry>
+                <cylinder radius="${wheel_radius}" length="${wheel_length}"/>
+            </geometry>
+            <material name="blue"/>
+        </visual>
+        <collision>
+            <geometry>
+                <cylinder radius="${wheel_radius}" length="${wheel_length}"/>
+            </geometry>
+        </collision>
+        <xacro:inertial_cylinder mass="${wheel_mass}" length="${wheel_length}" radius="${wheel_radius}">
+            <origin xyz="0 0 0" rpy="0 0 0"/>
+        </xacro:inertial_cylinder>
+    </link>
+    <!-- Joints -->
+    <joint name="chassis-base" type="fixed">
+        <parent link="base"/>
+        <child link="chassis"/>
+        <origin xyz="${chassis_joint_offset} 0 0"/>
+    </joint>
+    <joint name="left_back_wheel-base" type="continuous">
+        <parent link="base"/>
+        <child link="left_back_wheel"/>
+        <origin xyz="${backwheel_offset} ${leftwheel_offset} 0" rpy="${left_roll} 0 0"/>
+        <axis xyz="0 0 1"/>
+    </joint>
+    <joint name="right_back_wheel-base" type="continuous">
+        <parent link="base"/>
+        <child link="right_back_wheel"/>
+        <origin xyz="${backwheel_offset} ${rightwheel_offset} 0" rpy="${right_roll} 0 0"/>
+        <axis xyz="0 0 -1"/>
+    </joint>
+    <joint name="left_front_wheel-base" type="continuous">
+        <parent link="base"/>
+        <child link="left_front_wheel"/>
+        <origin xyz="${frontwheel_offset} ${leftwheel_offset} 0" rpy="${left_roll} 0 0"/>
+        <axis xyz="0 0 1"/>
+    </joint>
+    <joint name="right_front_wheel-base" type="continuous">
+        <parent link="base"/>
+        <child link="right_front_wheel"/>
+        <origin xyz="${frontwheel_offset} ${rightwheel_offset} 0" rpy="${right_roll} 0 0"/>
+        <axis xyz="0 0 -1"/>
+    </joint>
 </robot>

Commit message: added gazebo references

File: description/robot_core.xacro (robot description, xacro)
@@ -151,3 +151,19 @@
         <axis xyz="0 0 -1"/>
     </joint>
+    <!-- Gazebo References-->
+    <gazebo reference="chassis">
+        <material>Gazebo/White</material>
+    </gazebo>
+    <gazebo reference="left_back_wheel">
+        <material>Gazebo/Blue</material>
+     </gazebo>
+     <gazebo reference="right_back_wheel">
+        <material>Gazebo/Blue</material>
+     </gazebo>
+     <gazebo reference="left_front_wheel">
+        <material>Gazebo/Blue</material>
+     </gazebo>
+     <gazebo reference="right_front_wheel">
+        <material>Gazebo/Blue</material>
+     </gazebo>
 </robot>

Commit message: temporary fix frontwheels not appearing in Rviz (changed joint type)

File: description/robot_core.xacro (robot description, xacro)
@@ -139,5 +139,5 @@
         <axis xyz="0 0 -1"/>
     </joint>
-    <joint name="left_front_wheel-base" type="continuous">
+    <joint name="left_front_wheel-base" type="fixed">
         <parent link="base"/>
         <child link="left_front_wheel"/>
@@ -145,5 +145,5 @@
         <axis xyz="0 0 1"/>
     </joint>
-    <joint name="right_front_wheel-base" type="continuous">
+    <joint name="right_front_wheel-base" type="fixed">
         <parent link="base"/>
         <child link="right_front_wheel"/>
@@ -163,7 +163,11 @@
      <gazebo reference="left_front_wheel">
         <material>Gazebo/Blue</material>
+        <mu1 value="0.001"/>
+        <mu2 value="0.001"/>
      </gazebo>
      <gazebo reference="right_front_wheel">
         <material>Gazebo/Blue</material>
+        <mu1 value="0.001"/>
+        <mu2 value="0.001"/>
      </gazebo>
 </robot>

Commit message: added material red

File: description/robot_core.xacro (robot description, xacro)
@@ -35,4 +35,7 @@
     <material name="black">
         <color rgba="0 0 0 1"/>
+    </material>
+    <material name="red">
+        <color rgba="1 0 0 1"/>
     </material>
     <!-- links -->

Commit message: added footprint

File: description/robot_core.xacro (robot description, xacro)
@@ -41,4 +41,6 @@
     <!-- links -->
     <link name="base">
+    </link>
+    <link name="footprint">
     </link>
     <link name="chassis">
@@ -125,4 +127,9 @@
     </link>
     <!-- Joints -->
+    <joint name="footprint-base" type="fixed">
+        <parent link="base"/>
+        <child link="footprint"/>
+        <origin xyz="0 0 0" rpy="0 0 0"/>
+    </joint>
     <joint name="chassis-base" type="fixed">
         <parent link="base"/>
