Commit message: tried adding motor control

File: implement_bot/description/base_actual (4wheel).xacro (robot description, xacro)
@@ -53,46 +53,41 @@
         <xacro:scaled_origin x="${bot_pos_x}" y="${bot_pos_y}" z="${bot_pos_z}"/>
     </joint>
-    <!-- Caster link-joints -->
-    <xacro:macro name="caster_link_joint" params="pos_x axis">
-        <link name="${pos_x}_caster_link">
+    <!-- Motor link-joints -->
+    <xacro:macro name="motor_link_joint" params="pos_x axis">
+        <link name="${pos_x}_motor_link">
             <visual>
                 <geometry>
-                    <sphere radius="${actual_wheel_radius/2}"/>
+                    <cylinder radius="0.01" length="0.01"/>
                 </geometry>
-                <xacro:scaled_origin_rpy x="${-actual_shaft_length*2 -(actual_wheel_thickness/2)}" y="${actual_wheel_radius + actual_shaft_thickness}"  z="0.0" roll="0" pitch="0" yaw="0"/>
+                <xacro:scaled_origin_rpy x="${-actual_shaft_length*2 -(actual_wheel_thickness/2)}" y="${actual_wheel_radius + actual_shaft_thickness}"  z="${-actual_wheel_radius/2 + actual_shaft_thickness*2/3}" roll="0" pitch="0" yaw="0"/>
             </visual>
             <collision>
                 <geometry>
-                    <sphere radius="${actual_wheel_radius/2}"/>
+                    <cylinder radius="0.01" length="0.01"/>
                 </geometry>
-                <xacro:scaled_origin_rpy x="${-actual_shaft_length*2 -(actual_wheel_thickness/2)}" y="${actual_wheel_radius + actual_shaft_thickness}"  z="0.0" roll="0" pitch="0" yaw="0"/>
+                <origin xyz="0 0 0" rpy="0 ${pi/2} 0 "/>
             </collision>
-            <xacro:inertial_sphere mass="${wheel_mass}" radius="${actual_wheel_radius}">
-                <xacro:scaled_origin_rpy x="${-actual_shaft_length*2 -(actual_wheel_thickness/2)}" y="${actual_wheel_radius + actual_shaft_thickness}"  z="0.0" roll="0" pitch="0" yaw="0"/>
-            </xacro:inertial_sphere>
+            <xacro:inertial_cylinder mass="${wheel_mass}" length="${actual_wheel_thickness}" radius="${actual_wheel_radius}">
+                <origin xyz="0 0 0" rpy="0 ${pi/2} 0 "/>
+            </xacro:inertial_cylinder>
         </link>
         <xacro:if value="${pos_x == 'left'}">
-            <xacro:property name="wheel_x" value="${+(actual_bot_width/3)}"/>
+            <xacro:property name="wheel_x" value="${+(actual_bot_width/2) + actual_wheel_radius}"/>
             <xacro:property name="wheel_turn_x" value="0"/>
         </xacro:if>
         <xacro:if value="${pos_x == 'right'}">
-            <xacro:property name="wheel_x" value="${-(actual_bot_width/3)}"/>
+            <xacro:property name="wheel_x" value="${-(actual_bot_width/2) - actual_wheel_radius}"/>
             <xacro:property name="wheel_turn_x" value="${pi}"/>
         </xacro:if>
         <xacro:property name="wheel_turn_y" value="${pi/2}"/>
-        <joint name="${pos_x}_motor_joint" type="fixed">
+        <joint name="${pos_x}_motor_joint" type="continuous">
             <parent link="chassis_link"/>
-            <child link="${pos_x}_caster_link"/>
-            <xacro:scaled_origin_rpy x="${-(actual_bot_length/2 - actual_wheel_radius*2)}" y="${wheel_x}"  z="0" roll="0" pitch="${wheel_turn_x}" yaw="${wheel_turn_y}"/>
+            <child link="${pos_x}_motor_link"/>
+            <xacro:scaled_origin_rpy x="0.0" y="${wheel_x}"  z="${actual_wheel_radius/2}" roll="0" pitch="${wheel_turn_x}" yaw="${wheel_turn_y}"/>
             <axis xyz="${axis} 0 0"/>
         </joint>
-        <gazebo reference="${pos_x}_caster_link">
-            <material>Gazebo/Blue</material>
-            <mu1 value="0.01"/>
-            <mu2 value="0.01"/>
-         </gazebo>
     </xacro:macro>
-    <xacro:caster_link_joint pos_x="left" axis="1"/>
-    <xacro:caster_link_joint pos_x="right" axis="-1"/>
+    <xacro:motor_link_joint pos_x="left" axis="1"/>
+    <xacro:motor_link_joint pos_x="right" axis="-1"/>
     <!-- Wheel link-joints -->
     <xacro:macro name="wheel_link" params="pos_x pos_y">
@@ -119,4 +114,6 @@
         </link>
     </xacro:macro>
+    <xacro:wheel_link pos_x="left" pos_y="back"/>
+    <xacro:wheel_link pos_x="right" pos_y="back"/>
     <xacro:wheel_link pos_x="left" pos_y="front"/>
     <xacro:wheel_link pos_x="right" pos_y="front"/>
@@ -151,4 +148,6 @@
          </gazebo>
     </xacro:macro>
+    <xacro:wheel_joint pos_x="left" pos_y="back" axis="1"/>
+    <xacro:wheel_joint pos_x="right" pos_y="back" axis="-1"/>
     <xacro:wheel_joint pos_x="left" pos_y="front" axis="1"/>
     <xacro:wheel_joint pos_x="right" pos_y="front" axis="-1"/>

File: implement_bot/description/sensors.xacro (robot description, xacro)
@@ -1,5 +1,5 @@
 <?xml version="1.0"?>
 <robot xmlns:xacro="http://www.ros.org/wiki/xacro">
-    <link name="lidar_link">
+    <link name="ldlidar_link">
         <visual>
             <geometry>
@@ -21,5 +21,5 @@
     <joint name="lidar_link_joint" type="fixed">
         <parent link="chassis_link"/>
-        <child link="lidar_link"/>
+        <child link="ldlidar_link"/>
         <origin xyz="0.0 0.0 ${(scale_val* (actual_chassis_height + actual_storage_height + actual_top_height)) + 0.02}" rpy="0.0 0.0 0.0"/>
         <!-- <origin xyz="0.0 0.0 ${(scale_val* (actual_chassis_height) + 0.02)}" rpy="0.0 0.0 0.0"/> -->
@@ -27,5 +27,5 @@
     <link name="laser_frame" />
     <joint name="lidar_frame_joint" type="fixed">
-        <parent link="lidar_link"/>
+        <parent link="ldlidar_link"/>
         <child link="laser_frame"/>
         <origin xyz="0.0 0.0 ${scale_val* 0.0}" rpy="0.0 0.0 0.0"/>
