Commit message: sensor height fix(lowered)

File: implement_bot/description/sensors.xacro (robot description, xacro)
@@ -22,5 +22,6 @@
         <parent link="chassis_link"/>
         <child link="lidar_link"/>
-        <origin xyz="0.0 0.0 ${(scale_val* (actual_chassis_height + actual_storage_height + actual_top_height)) + 0.02}" rpy="0.0 0.0 0.0"/>
+        <!-- <origin xyz="0.0 0.0 ${(scale_val* (actual_chassis_height + actual_storage_height + actual_top_height)) + 0.02}" rpy="0.0 0.0 0.0"/> -->
+        <origin xyz="0.0 0.0 ${(scale_val* (actual_chassis_height) + 0.02)}" rpy="0.0 0.0 0.0"/>
     </joint>
     <link name="laser_frame" />

Commit message: leftover changes before merge

File: implement_bot/description/sensors.xacro (robot description, xacro)
@@ -22,6 +22,6 @@
         <parent link="chassis_link"/>
         <child link="lidar_link"/>
-        <!-- <origin xyz="0.0 0.0 ${(scale_val* (actual_chassis_height + actual_storage_height + actual_top_height)) + 0.02}" rpy="0.0 0.0 0.0"/> -->
-        <origin xyz="0.0 0.0 ${(scale_val* (actual_chassis_height) + 0.02)}" rpy="0.0 0.0 0.0"/>
+        <origin xyz="0.0 0.0 ${(scale_val* (actual_chassis_height + actual_storage_height + actual_top_height)) + 0.02}" rpy="0.0 0.0 0.0"/>
+        <!-- <origin xyz="0.0 0.0 ${(scale_val* (actual_chassis_height) + 0.02)}" rpy="0.0 0.0 0.0"/> -->
     </joint>
     <link name="laser_frame" />

Commit message: tried adding ir sensors

File: implement_bot/description/sensors.xacro (robot description, xacro)
@@ -58,3 +58,69 @@
         </sensor>
     </gazebo>
+    <xacro:macro name="range_link_joint" params="pos_x">
+        <link name="${pos_x}_range_link">
+            <visual>
+                <geometry>
+                    <box size="0.015 0.03 0.001"/>
+                </geometry>
+                <xacro:scaled_origin_rpy x="0.0" y="0.0"  z="0.0" roll="0" pitch="0" yaw="0"/>
+            </visual>
+            <collision>
+                <geometry>
+                    <box size="0.015 0.03 0.01"/>
+                </geometry>
+                <xacro:scaled_origin_rpy x="0.0" y="0.0"  z="0.0" roll="0" pitch="0" yaw="0"/>
+            </collision>
+            <xacro:inertial_box mass="0.001" x="0.0" y="0.0" z="0.0">
+            <origin xyz="0.0 0 0.0" rpy="-1 0 0"/>
+            </xacro:inertial_box>
+        </link>
+        <xacro:if value="${pos_x == 'left'}">
+            <xacro:property name="offset_x" value="${+(actual_bot_width/3)}"/>
+        </xacro:if>
+        <xacro:if value="${pos_x == 'right'}">
+            <xacro:property name="offset_x" value="${-(actual_bot_width/3)}"/>
+        </xacro:if>
+        <joint name="${pos_x}_range_joint" type="fixed">
+            <parent link="chassis_link"/>
+            <child link="${pos_x}_range_link"/>
+            <xacro:scaled_origin_rpy x="${(actual_bot_length/2) + smol_offset}" y="${offset_x}"  z="${actual_wheel_radius}" roll="0" pitch="0" yaw="0"/>
+            <axis xyz="0 0 0"/>
+        </joint>
+        <link name="${pos_x}_range_frame"/>
+        <joint name="${pos_x}_range_frame_joint" type="fixed">
+            <parent link="${pos_x}_range_link"/>
+            <child link="${pos_x}_range_frame"/>
+            <origin xyz="0.0 0.0 ${scale_val* 0.0}" rpy="0.0 0.0 0.0"/>
+        </joint>
+        <gazebo reference="${pos_x}_range_frame">
+        <sensor name="laser" type="ray">
+            <pose> 0 0 0 0 0 0 </pose>
+            <visualize>true</visualize>
+            <update_rate>10</update_rate>
+            <ray>
+                <scan>
+                    <horizontal>
+                        <samples>80</samples>
+                        <min_angle>0</min_angle>
+                        <max_angle>1</max_angle>
+                    </horizontal>
+                </scan>
+                <range>
+                    <min>0.1</min>
+                    <max>1</max>
+                </range>
+            </ray>
+            <plugin name="${pos_x}_range_sensGaz" filename="libgazebo_ros_ray_sensor.so">
+                <ros>
+                    <argument>~/out:=${pos_x}_range_frame</argument>
+                </ros>
+                <output_type>sensor_msgs/LaserScan</output_type>
+                <frame_name>${pos_x}range_frame</frame_name>
+            </plugin>
+        </sensor>
+        </gazebo>
+    </xacro:macro>
+    <xacro:range_link_joint pos_x="left"/>
+    <xacro:range_link_joint pos_x="right"/>
 </robot>

Commit message: imu sensor halfway done

File: implement_bot/description/sensors.xacro (robot description, xacro)
@@ -1,4 +1,5 @@
 <?xml version="1.0"?>
 <robot xmlns:xacro="http://www.ros.org/wiki/xacro">
+    <!-- Lidar Link -->
     <link name="ldlidar_link">
         <visual>
@@ -19,4 +20,5 @@
         </xacro:inertial_cylinder>
     </link>
+    <!-- Lidar Joint to Base Link -->
     <joint name="lidar_link_joint" type="fixed">
         <parent link="chassis_link"/>
@@ -25,5 +27,7 @@
         <!-- <origin xyz="0.0 0.0 ${(scale_val* (actual_chassis_height) + 0.02)}" rpy="0.0 0.0 0.0"/> -->
     </joint>
+    <!-- Lidar Frame that receives simulated data-->
     <link name="laser_frame" />
+    <!-- Joint to Lidar Link to Frame -->
     <joint name="lidar_frame_joint" type="fixed">
         <parent link="ldlidar_link"/>
@@ -31,4 +35,5 @@
         <origin xyz="0.0 0.0 ${scale_val* 0.0}" rpy="0.0 0.0 0.0"/>
     </joint>
+    <!-- Simulation Sensor for Laser Frame -->
     <gazebo reference="laser_frame">
         <sensor name="laser" type="ray">
@@ -58,4 +63,5 @@
         </sensor>
     </gazebo>
+    <!-- Macro for Ultrasonic Sensors -->
     <xacro:macro name="range_link_joint" params="pos_x">
         <link name="${pos_x}_range_link">
@@ -122,5 +128,44 @@
         </gazebo>
     </xacro:macro>
+    <!-- left ultrasonic sensor -->
     <xacro:range_link_joint pos_x="left"/>
+    <!-- right ultrasonic sensor -->
     <xacro:range_link_joint pos_x="right"/>
+    <!-- IMU Link -->
+    <link name="imu_link">
+        <visual>
+            <geometry>
+                <cylinder radius="0.01" length="0.01"/>
+            </geometry>
+            <origin xyz="0.0 0.0 0.0" rpy="0.0 0.0 ${pi}"/>
+        </visual>
+        <collision>
+            <geometry>
+                <cylinder radius="0.01" length="0.01"/>
+            </geometry>
+            <origin xyz="0.0 0.0 0.0" rpy="0.0 0.0 0.0"/>
+        </collision>
+        <xacro:inertial_cylinder mass="0.10" length="0.01" radius="0.01">
+                <xacro:scaled_origin_rpy x="0" y="0"  z="0" roll="0" pitch="0" yaw="0"/>
+        </xacro:inertial_cylinder>
+    </link>
+    <!-- IMU joint to base link -->
+    <joint name="imu_link_joint" type="fixed">
+        <parent link="chassis_link"/>
+        <child link="imu_link"/>
+        <origin xyz="0.0 0.0 {scale_val* 0.0}" rpy="0.0 0.0 0.0"/>
+    </joint>
+    <!-- IMU Frame for simulation-->
+    <link name="imu_frame" />
+    <!-- IMU Frame joint  -->
+    <joint name="imu_frame_joint" type="fixed">
+        <parent link="imu_link"/>
+        <child link="imu_frame"/>
+        <origin xyz="0.0 0.0 ${scale_val* 0.0}" rpy="0.0 0.0 0.0"/>
+    </joint>
+    <!-- IMU gazebo sensor -->
+    <gazebo reference="imu_frame">
+        <sensor name="imu_sensor" type="">
+        </sensor>
+    </gazebo>
 </robot>

Commit message: some stuffs got done before leaving

File: implement_bot/description/sensors.xacro (robot description, xacro)
@@ -33,5 +33,5 @@
         <parent link="ldlidar_link"/>
         <child link="laser_frame"/>
-        <origin xyz="0.0 0.0 ${scale_val* 0.0}" rpy="0.0 0.0 0.0"/>
+        <origin xyz="0.0 0.0 ${(scale_val)* 0.0}" rpy="0.0 0.0 0.0"/>
     </joint>
     <!-- Simulation Sensor for Laser Frame -->
@@ -154,5 +154,5 @@
         <parent link="chassis_link"/>
         <child link="imu_link"/>
-        <origin xyz="0.0 0.0 {scale_val* 0.0}" rpy="0.0 0.0 0.0"/>
+        <origin xyz="0.0 0.0 ${scale_val* 0.0}" rpy="0.0 0.0 0.0"/>
     </joint>
     <!-- IMU Frame for simulation-->
