Commit message: fixing robot description

File: implement_bot/description/gazebo_control.xacro (robot description, xacro)
@@ -1,54 +1,62 @@
 <?xml version="1.0"?>
-<!--Control Settings for Gazebo-->
 <robot xmlns:xacro="http://www.ros.org/wiki/xacro">
-    <!-- Gazebo References-->
-    <gazebo reference="chassis">
-        <material>Gazebo/White</material>
-    </gazebo>
-    <gazebo reference="left_back_wheel">
-        <material>Gazebo/Blue</material>
-     </gazebo>
-     <gazebo reference="right_back_wheel">
-        <material>Gazebo/Blue</material>
-     </gazebo>
-     <gazebo reference="left_front_wheel">
-        <material>Gazebo/Blue</material>
-        <mu1 value="0.0"/>
-        <mu2 value="0.0"/>
-     </gazebo>
-     <gazebo reference="right_front_wheel">
-        <material>Gazebo/Blue</material>
-        <mu1 value="0.0"/>
-        <mu2 value="0.0"/>
-     </gazebo>
-     <!-- Gazebo drive system -->
+    <!-- For Gazebo Hardware Interface -->
+    <ros2_control name="GazBotSys" type="system">
+        <hardware>
+            <plugin>gazebo_ros2_control/GazeboSystem</plugin>
+        </hardware>
+        <joint name='left_back_wheel_joint'>
+            <command_interface name="velocity">
+                <param name="min">-10</param>
+                <param name="max">10</param>
+            </command_interface>
+            <state_interface name="velocity"/>
+            <state_interface name="position"/>
+        </joint>
+        <joint name='right_back_wheel_joint'>
+            <command_interface name="velocity">
+                <param name="min">-10</param>
+                <param name="max">10</param>
+            </command_interface>
+            <state_interface name="velocity"/>
+            <state_interface name="position"/>
+        </joint>
+        <joint name='left_front_wheel_joint'>
+            <command_interface name="velocity">
+                <param name="min">-10</param>
+                <param name="max">10</param>
+            </command_interface>
+            <state_interface name="velocity"/>
+            <state_interface name="position"/>
+        </joint>
+        <joint name='right_front_wheel_joint'>
+            <command_interface name="velocity">
+                <param name="min">-10</param>
+                <param name="max">10</param>
+            </command_interface>
+            <state_interface name="velocity"/>
+            <state_interface name="position"/>
+        </joint>
+        <joint name='left_motor_joint'>
+            <command_interface name="velocity">
+                <param name="min">-10</param>
+                <param name="max">10</param>
+            </command_interface>
+            <state_interface name="velocity"/>
+            <state_interface name="position"/>
+        </joint>
+        <joint name='right_motor_joint'>
+            <command_interface name="velocity">
+                <param name="min">-10</param>
+                <param name="max">10</param>
+            </command_interface>
+            <state_interface name="velocity"/>
+            <state_interface name="position"/>
+        </joint>
+    </ros2_control>
+    <!-- For Gazebo Simulation of ROS2 Control -->
     <gazebo>
-        <plugin name="drive" filename="libgazebo_ros_diff_drive.so">
-            <!-- Wheel information -->
-            <left_joint>left_back_wheel_joint</left_joint>
-            <right_joint>right_back_wheel_joint</right_joint>
-            <wheel_separation>0.35</wheel_separation>
-            <wheel_diameter>0.1</wheel_diameter>
-            <!-- Limits -->
-            <max_wheel_torque>200</max_wheel_torque>
-            <max_wheel_acceleration>10.0</max_wheel_acceleration>
-            <!-- Output -->
-            <odometry_frame>odom</odometry_frame>
-            <robot_base_frame>base_link</robot_base_frame>
-            <publish_odom>true</publish_odom>
-            <publish_odom_tf>true</publish_odom_tf>
-            <publish_wheel_tf>true</publish_wheel_tf>
-        </plugin>
-    </gazebo>
-    <!-- Gazebo requires the use of plugins to interact with other systems such as ROS. -->
-    <!-- This plugin will publish the joint_states for the selected joints
-            (which robot_state_publisher can then use to broadcast the approprate tf). -->
-    <gazebo>
-        <plugin name="gazebo_ros_joint_state_publisher" filename="libgazebo_ros_joint_state_publisher.so">
-            <update_rate>20</update_rate>
-            <joint_name>left_back_wheel_joint</joint_name>
-            <joint_name>right_back_wheel_joint</joint_name>
-            <joint_name>left_front_wheel_joint</joint_name>
-            <joint_name>right_front_wheel_joint</joint_name>
+        <plugin name="ros2_controller" filename="libgazebo_ros2_control.so">
+            <parameters>$(find implement_bot)/config/gazebo_controller_params.yaml</parameters>
         </plugin>
     </gazebo>

File: implement_bot/description/main_urdf.xacro (robot description, xacro)
@@ -2,5 +2,5 @@
 <!-- loaded urdf file for robot-->
 <robot xmlns:xacro="http://www.ros.org/wiki/xacro"  name="robot1">
-    <xacro:property name="use_ros2_control" value="true"/>
+    <xacro:property name="use_ros2_control" value="false"/>
     <xacro:if value="${use_ros2_control}">
         <xacro:include filename="ros2_control.xacro"/>

File: implement_bot/description/ros2_control.xacro (robot description, xacro)
@@ -1,6 +1,6 @@
 <?xml version="1.0"?>
 <robot xmlns:xacro="http://www.ros.org/wiki/xacro">
-    <!-- For Gazebo Hardware Interface -->
-    <ros2_control name="GazBotSys" type="system">
+    <!-- For Real Hardware Interface -->
+    <ros2_control name="ActBotSys" type="system">
         <hardware>
             <plugin>gazebo_ros2_control/GazeboSystem</plugin>
@@ -55,9 +55,3 @@
         </joint>
     </ros2_control>
-    <!-- For Gazebo Simulation of ROS2 Control -->
-    <gazebo>
-        <plugin name="ros2_controller" filename="libgazebo_ros2_control.so">
-            <parameters>$(find implement_bot)/config/gazebo_controller_params.yaml</parameters>
-        </plugin>
-    </gazebo>
 </robot>

Commit message: added ros2 control

File: implement_bot/description/gazebo_control.xacro (robot description, xacro)
@@ -6,21 +6,5 @@
             <plugin>gazebo_ros2_control/GazeboSystem</plugin>
         </hardware>
-        <joint name='left_back_wheel_joint'>
-            <command_interface name="velocity">
-                <param name="min">-10</param>
-                <param name="max">10</param>
-            </command_interface>
-            <state_interface name="velocity"/>
-            <state_interface name="position"/>
-        </joint>
-        <joint name='right_back_wheel_joint'>
-            <command_interface name="velocity">
-                <param name="min">-10</param>
-                <param name="max">10</param>
-            </command_interface>
-            <state_interface name="velocity"/>
-            <state_interface name="position"/>
-        </joint>
-        <joint name='left_front_wheel_joint'>
+                <joint name='left_front_wheel_joint'>
             <command_interface name="velocity">
                 <param name="min">-10</param>
@@ -38,26 +22,4 @@
             <state_interface name="position"/>
         </joint>
-        <joint name='left_motor_joint'>
-            <command_interface name="velocity">
-                <param name="min">-10</param>
-                <param name="max">10</param>
-            </command_interface>
-            <state_interface name="velocity"/>
-            <state_interface name="position"/>
-        </joint>
-        <joint name='right_motor_joint'>
-            <command_interface name="velocity">
-                <param name="min">-10</param>
-                <param name="max">10</param>
-            </command_interface>
-            <state_interface name="velocity"/>
-            <state_interface name="position"/>
-        </joint>
     </ros2_control>
-    <!-- For Gazebo Simulation of ROS2 Control -->
-    <gazebo>
-        <plugin name="ros2_controller" filename="libgazebo_ros2_control.so">
-            <parameters>$(find implement_bot)/config/gazebo_controller_params.yaml</parameters>
-        </plugin>
-    </gazebo>
 </robot>

File: implement_bot/description/ros2_control.xacro (robot description, xacro)
@@ -4,5 +4,16 @@
     <ros2_control name="ActBotSys" type="system">
         <hardware>
-            <plugin>gazebo_ros2_control/GazeboSystem</plugin>
+            <plugin>diffdrive_arduino/DiffDriveArduinoHardware</plugin>
+            <param name="left_wheel_name">left_wheel_joint</param>
+            <param name="right_wheel_name">right_wheel_joint</param>
+            <param name="loop_rate">30</param>
+            <param name="device">/dev/serial/by-path/platform-fd500000.pcie-pci-0000:01:00.0-usb-0:1.3:1.0-port0</param>
+            <param name="baud_rate">57600</param>
+            <param name="timeout_ms">1000</param>
+            <param name="enc_counts_per_rev">3000</param>
+            <param name="pid_p">20</param>
+            <param name="pid_d">12</param>
+            <param name="pid_i">0</param>
+            <param name="pid_o">50</param>
         </hardware>
         <joint name='left_back_wheel_joint'>

Commit message: working hardware interface

File: implement_bot/description/gazebo_control.xacro (robot description, xacro)
@@ -6,5 +6,5 @@
             <plugin>gazebo_ros2_control/GazeboSystem</plugin>
         </hardware>
-                <joint name='left_front_wheel_joint'>
+        <joint name='left_front_wheel_joint'>
             <command_interface name="velocity">
                 <param name="min">-10</param>

File: implement_bot/description/main_urdf.xacro (robot description, xacro)
@@ -2,5 +2,5 @@
 <!-- loaded urdf file for robot-->
 <robot xmlns:xacro="http://www.ros.org/wiki/xacro"  name="robot1">
-    <xacro:property name="use_ros2_control" value="false"/>
+    <xacro:property name="use_ros2_control" value="true"/>
     <xacro:if value="${use_ros2_control}">
         <xacro:include filename="ros2_control.xacro"/>

File: implement_bot/description/ros2_control.xacro (robot description, xacro)
@@ -4,9 +4,10 @@
     <ros2_control name="ActBotSys" type="system">
         <hardware>
-            <plugin>diffdrive_arduino/DiffDriveArduinoHardware</plugin>
-            <param name="left_wheel_name">left_wheel_joint</param>
-            <param name="right_wheel_name">right_wheel_joint</param>
+            <plugin>DiffBotHardwareSystem</plugin>
+            <param name="left_wheel_name">left_front_wheel_joint</param>
+            <param name="right_wheel_name">right_front_wheel_joint</param>
             <param name="loop_rate">30</param>
-            <param name="device">/dev/serial/by-path/platform-fd500000.pcie-pci-0000:01:00.0-usb-0:1.3:1.0-port0</param>
+            <!-- <param name="device">/dev/serial/by-path/platform-fd500000.pcie-pci-0000:01:00.0-usb-0:1.3:1.0-port0</param> -->
+            <param name="device">/dev/ttyUSB0</param>
             <param name="baud_rate">57600</param>
             <param name="timeout_ms">1000</param>
@@ -17,52 +18,14 @@
             <param name="pid_o">50</param>
         </hardware>
-        <joint name='left_back_wheel_joint'>
-            <command_interface name="velocity">
-                <param name="min">-10</param>
-                <param name="max">10</param>
-            </command_interface>
-            <state_interface name="velocity"/>
-            <state_interface name="position"/>
-        </joint>
-        <joint name='right_back_wheel_joint'>
-            <command_interface name="velocity">
-                <param name="min">-10</param>
-                <param name="max">10</param>
-            </command_interface>
-            <state_interface name="velocity"/>
-            <state_interface name="position"/>
-        </joint>
-        <joint name='left_front_wheel_joint'>
-            <command_interface name="velocity">
-                <param name="min">-10</param>
-                <param name="max">10</param>
-            </command_interface>
+        <!-- <joint name='left_front_wheel_joint'>
+            <command_interface name="velocity"/>
             <state_interface name="velocity"/>
             <state_interface name="position"/>
         </joint>
         <joint name='right_front_wheel_joint'>
-            <command_interface name="velocity">
-                <param name="min">-10</param>
-                <param name="max">10</param>
-            </command_interface>
+            <command_interface name="velocity"/>
             <state_interface name="velocity"/>
             <state_interface name="position"/>
-        </joint>
-        <joint name='left_motor_joint'>
-            <command_interface name="velocity">
-                <param name="min">-10</param>
-                <param name="max">10</param>
-            </command_interface>
-            <state_interface name="velocity"/>
-            <state_interface name="position"/>
-        </joint>
-        <joint name='right_motor_joint'>
-            <command_interface name="velocity">
-                <param name="min">-10</param>
-                <param name="max">10</param>
-            </command_interface>
-            <state_interface name="velocity"/>
-            <state_interface name="position"/>
-        </joint>
+        </joint> -->
     </ros2_control>
 </robot>
