Commit message: moved gazebo sensors

File: implement_bot/description/gazebo_control.xacro (robot description, xacro)
@@ -32,3 +32,149 @@
         </plugin>
     </gazebo>
+    <!-- Lidar Frame that receives simulated data-->
+    <link name="laser_frame" />
+    <!-- Joint to Lidar Link to Frame -->
+    <joint name="lidar_frame_joint" type="fixed">
+        <parent link="ldlidar_link"/>
+        <child link="laser_frame"/>
+        <origin xyz="0.0 0.0 ${(scale_val)* 0.0}" rpy="0.0 0.0 0.0"/>
+    </joint>
+    <!-- Simulation Sensor for Laser Frame -->
+    <gazebo reference="laser_frame">
+        <sensor name="laser" type="ray">
+            <pose> 0 0 0 0 0 0 </pose>
+            <visualize>true</visualize>
+            <update_rate>10</update_rate>
+            <ray>
+                <scan>
+                    <horizontal>
+                        <samples>720</samples>
+                        <min_angle>-3.14</min_angle>
+                        <max_angle>3.14</max_angle>
+                    </horizontal>
+                </scan>
+                <range>
+                    <min>0.1</min>
+                    <max>12</max>
+                </range>
+            </ray>
+            <plugin name="lidar_gazebo" filename="libgazebo_ros_ray_sensor.so">
+                <ros>
+                    <argument>~/out:=gazebo/scan</argument>
+                </ros>
+                <output_type>sensor_msgs/LaserScan</output_type>
+                <frame_name>laser_frame</frame_name>
+            </plugin>
+        </sensor>
+    </gazebo>
+    <!-- Macro for Ultrasonic Sensors -->
+    <xacro:macro name="range_link_joint" params="pos_x">
+        <gazebo reference="${pos_x}_range_frame">
+            <sensor name="${pos_x}_us_sensor" type="ray">
+                <pose> 0 0 0 0 0 0 </pose>
+                <visualize>true</visualize>
+                <update_rate>10</update_rate>
+                <ray>
+                    <scan>
+                        <horizontal>
+                            <samples>80</samples>
+                            <min_angle>-0.45</min_angle>
+                            <max_angle>0.45</max_angle>
+                        </horizontal>
+                    </scan>
+                    <range>
+                        <min>0.1</min>
+                        <max>1</max>
+                    </range>
+                </ray>
+                <plugin name="${pos_x}_range_sensGaz" filename="libgazebo_ros_ray_sensor.so">
+                    <ros>
+                        <argument>~/out:=gazebo/${pos_x}_range_frame</argument>
+                    </ros>
+                    <output_type>sensor_msgs/LaserScan</output_type>
+                    <frame_name>${pos_x}range_frame</frame_name>
+                </plugin>
+            </sensor>
+        </gazebo>
+    </xacro:macro>
+    <!-- left ultrasonic sensor -->
+    <xacro:range_link_joint pos_x="left"/>
+    <!-- right ultrasonic sensor -->
+    <xacro:range_link_joint pos_x="right"/>
+    <!-- IMU Frame for simulation-->
+    <link name="imu_frame" />
+    <!-- IMU Frame joint  -->
+    <joint name="imu_frame_joint" type="fixed">
+        <parent link="imu_link"/>
+        <child link="imu_frame"/>
+        <origin xyz="0.0 0.0 ${scale_val* 0.0}" rpy="0.0 0.0 0.0"/>
+    </joint>
+    <!-- IMU gazebo sensor -->
+    <gazebo reference="imu_frame">
+        <sensor name="imu_sensor" type="imu">
+        <plugin filename="libgazebo_ros_imu_sensor.so" name="imu_plugin">
+            <ros>
+                <remapping>~/out:=gazebo/imu_odom</remapping>
+            </ros>
+            <initial_orientation_as_reference>false</initial_orientation_as_reference>
+            </plugin>
+            <always_on>true</always_on>
+            <update_rate>100</update_rate>
+            <visualize>true</visualize>
+            <imu>
+            <angular_velocity>
+                <x>
+                <noise type="gaussian">
+                    <mean>0.0</mean>
+                    <stddev>2e-4</stddev>
+                    <bias_mean>0.0000075</bias_mean>
+                    <bias_stddev>0.0000008</bias_stddev>
+                </noise>
+                </x>
+                <y>
+                <noise type="gaussian">
+                    <mean>0.0</mean>
+                    <stddev>2e-4</stddev>
+                    <bias_mean>0.0000075</bias_mean>
+                    <bias_stddev>0.0000008</bias_stddev>
+                </noise>
+                </y>
+                <z>
+                <noise type="gaussian">
+                    <mean>0.0</mean>
+                    <stddev>2e-4</stddev>
+                    <bias_mean>0.0000075</bias_mean>
+                    <bias_stddev>0.0000008</bias_stddev>
+                </noise>
+                </z>
+            </angular_velocity>
+            <linear_acceleration>
+                <x>
+                <noise type="gaussian">
+                    <mean>0.0</mean>
+                    <stddev>1.7e-2</stddev>
+                    <bias_mean>0.1</bias_mean>
+                    <bias_stddev>0.001</bias_stddev>
+                </noise>
+                </x>
+                <y>
+                <noise type="gaussian">
+                    <mean>0.0</mean>
+                    <stddev>1.7e-2</stddev>
+                    <bias_mean>0.1</bias_mean>
+                    <bias_stddev>0.001</bias_stddev>
+                </noise>
+                </y>
+                <z>
+                <noise type="gaussian">
+                    <mean>0.0</mean>
+                    <stddev>1.7e-2</stddev>
+                    <bias_mean>0.1</bias_mean>
+                    <bias_stddev>0.001</bias_stddev>
+                </noise>
+                </z>
+            </linear_acceleration>
+            </imu>
+        </sensor>
+    </gazebo>
 </robot>

File: implement_bot/description/sensors.xacro (robot description, xacro)
@@ -27,40 +27,4 @@
         <!-- <origin xyz="0.0 0.0 ${(scale_val* (actual_chassis_height) + 0.02)}" rpy="0.0 0.0 0.0"/> -->
     </joint>
-    <!-- Lidar Frame that receives simulated data-->
-    <link name="laser_frame" />
-    <!-- Joint to Lidar Link to Frame -->
-    <joint name="lidar_frame_joint" type="fixed">
-        <parent link="ldlidar_link"/>
-        <child link="laser_frame"/>
-        <origin xyz="0.0 0.0 ${(scale_val)* 0.0}" rpy="0.0 0.0 0.0"/>
-    </joint>
-    <!-- Simulation Sensor for Laser Frame -->
-    <gazebo reference="laser_frame">
-        <sensor name="laser" type="ray">
-            <pose> 0 0 0 0 0 0 </pose>
-            <visualize>true</visualize>
-            <update_rate>10</update_rate>
-            <ray>
-                <scan>
-                    <horizontal>
-                        <samples>720</samples>
-                        <min_angle>-3.14</min_angle>
-                        <max_angle>3.14</max_angle>
-                    </horizontal>
-                </scan>
-                <range>
-                    <min>0.1</min>
-                    <max>12</max>
-                </range>
-            </ray>
-            <plugin name="lidar_gazebo" filename="libgazebo_ros_ray_sensor.so">
-                <ros>
-                    <argument>~/out:=gazebo/scan</argument>
-                </ros>
-                <output_type>sensor_msgs/LaserScan</output_type>
-                <frame_name>laser_frame</frame_name>
-            </plugin>
-        </sensor>
-    </gazebo>
     <!-- Macro for Ultrasonic Sensors -->
     <xacro:macro name="range_link_joint" params="pos_x">
@@ -100,31 +64,4 @@
             <origin xyz="0.0 0.0 ${scale_val* 0.0}" rpy="0.0 0.0 0.0"/>
         </joint>
-        <gazebo reference="${pos_x}_range_frame">
-        <sensor name="${pos_x}_us_sensor" type="ray">
-            <pose> 0 0 0 0 0 0 </pose>
-            <visualize>true</visualize>
-            <update_rate>10</update_rate>
-            <ray>
-                <scan>
-                    <horizontal>
-                        <samples>80</samples>
-                        <min_angle>-0.45</min_angle>
-                        <max_angle>0.45</max_angle>
-                    </horizontal>
-                </scan>
-                <range>
-                    <min>0.1</min>
-                    <max>1</max>
-                </range>
-            </ray>
-            <plugin name="${pos_x}_range_sensGaz" filename="libgazebo_ros_ray_sensor.so">
-                <ros>
-                    <argument>~/out:=gazebo/${pos_x}_range_frame</argument>
-                </ros>
-                <output_type>sensor_msgs/LaserScan</output_type>
-                <frame_name>${pos_x}range_frame</frame_name>
-            </plugin>
-        </sensor>
-        </gazebo>
     </xacro:macro>
     <!-- left ultrasonic sensor -->
@@ -156,79 +93,3 @@
         <origin xyz="0.0 0.0 ${scale_val* 0.0}" rpy="0.0 0.0 0.0"/>
     </joint>
-    <!-- IMU Frame for simulation-->
-    <link name="imu_frame" />
-    <!-- IMU Frame joint  -->
-    <joint name="imu_frame_joint" type="fixed">
-        <parent link="imu_link"/>
-        <child link="imu_frame"/>
-        <origin xyz="0.0 0.0 ${scale_val* 0.0}" rpy="0.0 0.0 0.0"/>
-    </joint>
-    <!-- IMU gazebo sensor -->
-    <gazebo reference="imu_frame">
-        <sensor name="imu_sensor" type="imu">
-        <plugin filename="libgazebo_ros_imu_sensor.so" name="imu_plugin">
-            <ros>
-                <remapping>~/out:=gazebo/imu_odom</remapping>
-            </ros>
-            <initial_orientation_as_reference>false</initial_orientation_as_reference>
-            </plugin>
-            <always_on>true</always_on>
-            <update_rate>100</update_rate>
-            <visualize>true</visualize>
-            <imu>
-            <angular_velocity>
-                <x>
-                <noise type="gaussian">
-                    <mean>0.0</mean>
-                    <stddev>2e-4</stddev>
-                    <bias_mean>0.0000075</bias_mean>
-                    <bias_stddev>0.0000008</bias_stddev>
-                </noise>
-                </x>
-                <y>
-                <noise type="gaussian">
-                    <mean>0.0</mean>
-                    <stddev>2e-4</stddev>
-                    <bias_mean>0.0000075</bias_mean>
-                    <bias_stddev>0.0000008</bias_stddev>
-                </noise>
-                </y>
-                <z>
-                <noise type="gaussian">
-                    <mean>0.0</mean>
-                    <stddev>2e-4</stddev>
-                    <bias_mean>0.0000075</bias_mean>
-                    <bias_stddev>0.0000008</bias_stddev>
-                </noise>
-                </z>
-            </angular_velocity>
-            <linear_acceleration>
-                <x>
-                <noise type="gaussian">
-                    <mean>0.0</mean>
-                    <stddev>1.7e-2</stddev>
-                    <bias_mean>0.1</bias_mean>
-                    <bias_stddev>0.001</bias_stddev>
-                </noise>
-                </x>
-                <y>
-                <noise type="gaussian">
-                    <mean>0.0</mean>
-                    <stddev>1.7e-2</stddev>
-                    <bias_mean>0.1</bias_mean>
-                    <bias_stddev>0.001</bias_stddev>
-                </noise>
-                </y>
-                <z>
-                <noise type="gaussian">
-                    <mean>0.0</mean>
-                    <stddev>1.7e-2</stddev>
-                    <bias_mean>0.1</bias_mean>
-                    <bias_stddev>0.001</bias_stddev>
-                </noise>
-                </z>
-            </linear_acceleration>
-            </imu>
-        </sensor>
-    </gazebo>
 </robot>

Commit message: moved gazebo sensors

File: implement_bot/description/gazebo_control.xacro (robot description, xacro)
@@ -70,4 +70,10 @@
     <!-- Macro for Ultrasonic Sensors -->
     <xacro:macro name="range_link_joint" params="pos_x">
+        <link name="${pos_x}_range_frame"/>
+        <joint name="${pos_x}_range_frame_joint" type="fixed">
+            <parent link="${pos_x}_range_link"/>
+            <child link="${pos_x}_range_frame"/>
+            <origin xyz="0.0 0.0 ${scale_val* 0.0}" rpy="0.0 0.0 0.0"/>
+        </joint>
         <gazebo reference="${pos_x}_range_frame">
             <sensor name="${pos_x}_us_sensor" type="ray">

File: implement_bot/description/sensors.xacro (robot description, xacro)
@@ -58,10 +58,4 @@
             <axis xyz="0 0 0"/>
         </joint>
-        <link name="${pos_x}_range_frame"/>
-        <joint name="${pos_x}_range_frame_joint" type="fixed">
-            <parent link="${pos_x}_range_link"/>
-            <child link="${pos_x}_range_frame"/>
-            <origin xyz="0.0 0.0 ${scale_val* 0.0}" rpy="0.0 0.0 0.0"/>
-        </joint>
     </xacro:macro>
     <!-- left ultrasonic sensor -->

Commit message: gazebo sim stuff

File: implement_bot/description/gazebo_control.xacro (robot description, xacro)
@@ -1,4 +1,6 @@
 <?xml version="1.0"?>
 <robot xmlns:xacro="http://www.ros.org/wiki/xacro">
+    <!-- Properties xacro-->
+    <xacro:include filename="base_properties.xacro"/>
     <!-- For Gazebo Hardware Interface -->
     <ros2_control name="GazBotSys" type="system">
@@ -27,7 +29,7 @@
         <plugin name="ros2_controller" filename="libgazebo_ros2_control.so">
             <parameters>$(find implement_bot)/config/gazebo_controller_params.yaml</parameters>
-            <ros>
+            <!-- <ros>
                 <remapping>~/odom:=gazebo/wheel_odom</remapping>
-            </ros>
+            </ros> -->
         </plugin>
     </gazebo>
@@ -38,5 +40,5 @@
         <parent link="ldlidar_link"/>
         <child link="laser_frame"/>
-        <origin xyz="0.0 0.0 ${(scale_val)* 0.0}" rpy="0.0 0.0 0.0"/>
+        <origin xyz="0.0 0.0 ${scale_val * 0.0 + 0}" rpy="0.0 0.0 0.0"/>
     </joint>
     <!-- Simulation Sensor for Laser Frame -->
