Commit message: finished setting up hardware interfaces. Still need to add read functions

File: implement_bot/description/main_urdf.xacro (robot description, xacro)
@@ -7,5 +7,5 @@
     </xacro:if>
     <xacro:unless value="${use_ros2_control}">
-        <xacro:include filename="gazebo_control.xacro"/>
+        <!-- <xacro:include filename="gazebo_control.xacro"/> -->
     </xacro:unless>
     <xacro:include filename="base_actual.xacro"/>

File: implement_bot/description/ros2_control.xacro (robot description, xacro)
@@ -4,5 +4,5 @@
     <ros2_control name="ActBotSys" type="system">
         <hardware>
-            <plugin>DiffBotHardwareSystem</plugin>
+            <plugin>BotHardwareSystem</plugin>
             <param name="left_wheel_name">left_front_wheel_joint</param>
             <param name="right_wheel_name">right_front_wheel_joint</param>
@@ -17,15 +17,8 @@
             <param name="pid_i">0</param>
             <param name="pid_o">50</param>
+            <param name="left_range_name">left_range</param>
+            <param name="right_range_name">right_range</param>
+            <param name="imu_name">imu</param>
         </hardware>
-         <joint name='left_front_wheel_joint'>
-            <command_interface name="velocity"/>
-            <state_interface name="velocity"/>
-            <state_interface name="position"/>
-        </joint>
-        <joint name='right_front_wheel_joint'>
-            <command_interface name="velocity"/>
-            <state_interface name="velocity"/>
-            <state_interface name="position"/>
-        </joint>
     </ros2_control>
 </robot>
