Commit message: nav updates

File: implement_bot/description/base_properties.xacro (robot description, xacro)
@@ -20,7 +20,7 @@
     <xacro:property name="actual_bot_length" value="0.4572"/>
     <xacro:property name="actual_chassis_height" value="0.2286"/>
-    <xacro:property name="chassis_mass" value="5.0"/>
+    <xacro:property name="chassis_mass" value="50.0"/>
     <xacro:property name="actual_storage_height" value="0.4572"/>
-    <xacro:property name="storage_mass" value="10.0"/>
+    <xacro:property name="storage_mass" value="150.0"/>
     <xacro:property name="actual_top_height" value="0.1524"/>
     <xacro:property name="top_mass" value="10.0"/>

File: implement_bot/description/ros2_control.xacro (robot description, xacro)
@@ -7,5 +7,5 @@
             <param name="left_wheel_name">left_front_wheel_joint</param>
             <param name="right_wheel_name">right_front_wheel_joint</param>
-            <param name="loop_rate">30</param>
+            <param name="loop_rate">40</param>
             <param name="device">/dev/serial/by-path/platform-fd500000.pcie-pci-0000:01:00.0-usb-0:1.2:1.0-port0</param>
             <!-- <param name="device">/dev/serial1</param> -->
