Commit message: fixed actual xacro (w/o  actual values yet)

File: implement_bot/description/base_actual.xacro (robot description, xacro)
@@ -4,122 +4,98 @@
 <!-- call xacro-->
 <robot xmlns:xacro="http://www.ros.org/wiki/xacro">
-    <!-- Inertial xacro-->
+    <!-- Properties xacro-->
     <xacro:include filename="base_properties.xacro"/>
-    <!-- links -->
+    <!-- World link-joints -->
     <link name="base_link">
     </link>
     <link name="base_footprint">
     </link>
+    <joint name="base_joint" type="fixed">
+        <parent link="base_footprint"/>
+        <child link="base_link"/>
+        <origin xyz="0 0 0" rpy="0 0 0"/>
+    </joint>
+    <!-- <link name="odom">
+    </link>
+    <joint name="base_odom" type="fixed">
+        <parent link="base_footprint"/>
+        <child link="odom"/>
+        <origin xyz="0 0 0" rpy="0 0 0"/>
+    </joint> -->
+    <!-- Body link-joints -->
     <link name="chassis_link">
         <visual>
-            <origin xyz="${chassis_link_offset} 0 ${chassis_height_offset}"/>
             <geometry>
-                <mesh filename="package://bot/description/meshes/model-base_part.dae"/>
+                <mesh filename="package://bot/description/meshes/model-chassis_part.dae" scale="${scale}"/>
             </geometry>
-        </visual>
-        <collision>
-            <origin xyz="${chassis_link_offset} 0 ${chassis_height_offset}"/>
-            <geometry>
-                <mesh filename="package://bot/description/meshes/model-base_part.dae"/>
-            </geometry>
-        </collision>
-        <xacro:inertial_box mass="${chassis_mass}" x="${chassis_base}" y="${chassis_base}" z="${chassis_height}">
-            <origin xyz="${chassis_link_offset} 0 ${chassis_height_offset}" rpy="0 0 0"/>
-        </xacro:inertial_box>
-    </link>
-    <link name="left_back_wheel">
-        <visual>
-            <geometry>
-                <mesh filename="package://bot/description/meshes/model-wheel_part_curve.dae"/>
-            </geometry>
+            <xacro:scaled_origin x="0.0" y="0.0" z="0.0"/>
         </visual>
         <collision>
             <geometry>
-                <mesh filename="package://bot/description/meshes/model-wheel_part_curve.dae"/>
+                <mesh filename="package://bot/description/meshes/model-chassis_part.dae" scale="${scale}"/>
             </geometry>
+            <xacro:scaled_origin x="0.0" y="0.0" z="0.0"/>
         </collision>
-        <xacro:inertial_cylinder mass="${wheel_mass}" length="${wheel_length}" radius="${wheel_radius}">
-            <origin xyz="0 0 0" rpy="0 0 0"/>
-        </xacro:inertial_cylinder>
+        <xacro:inertial_box mass="${chassis_mass}" x="${actual_bot_width}" y="${actual_bot_length}" z="${actual_chassis_height}">
+            <!-- <origin xyz="0 0 0" rpy="0 0 0"/> -->
+            <xacro:scaled_origin_rpy x="0" y="0"  z="0" roll="0" pitch="0" yaw="0"/>
+        </xacro:inertial_box>
     </link>
-    <link name="right_back_wheel">
-        <visual>
-            <geometry>
-                <mesh filename="package://bot/description/meshes/model-wheel_part_curve.dae"/>
-            </geometry>
-        </visual>
-        <collision>
-            <geometry>
-                <mesh filename="package://bot/description/meshes/model-wheel_part_curve.dae"/>
-            </geometry>
-        </collision>
-        <xacro:inertial_cylinder mass="${wheel_mass}" length="${wheel_length}" radius="${wheel_radius}">
-            <origin xyz="0 0 0" rpy="0 0 0"/>
-        </xacro:inertial_cylinder>
-    </link>
-    <link name="left_front_wheel">
-        <visual>
-            <geometry>
-                <mesh filename="package://bot/description/meshes/model-wheel_part_curve.dae"/>
-            </geometry>
-        </visual>
-        <collision>
-            <geometry>
-                <mesh filename="package://bot/description/meshes/model-wheel_part_curve.dae"/>
-            </geometry>
-        </collision>
-        <xacro:inertial_cylinder mass="${wheel_mass}" length="${wheel_length}" radius="${wheel_radius}">
-            <origin xyz="0 0 0" rpy="0 0 0"/>
-        </xacro:inertial_cylinder>
-    </link>
-    <link name="right_front_wheel">
-        <visual>
-            <geometry>
-                <mesh filename="package://bot/description/meshes/model-wheel_part_curve.dae"/>
-            </geometry>
-        </visual>
-        <collision>
-            <geometry>
-                <mesh filename="package://bot/description/meshes/model-wheel_part_curve.dae"/>
-            </geometry>
-        </collision>
-        <xacro:inertial_cylinder mass="${wheel_mass}" length="${wheel_length}" radius="${wheel_radius}">
-            <origin xyz="0 0 0" rpy="0 0 0"/>
-        </xacro:inertial_cylinder>
-    </link>
-    <!-- Joints -->
-    <joint name="footprint-base" type="fixed">
-        <parent link="base"/>
-        <child link="footprint"/>
-        <origin xyz="0 0 0" rpy="0 0 0"/>
+    <joint name="chassis_joint" type="fixed">
+        <parent link="base_link"/>
+        <child link="chassis_link"/>
+        <xacro:scaled_origin x="0.0" y="0.0" z="0.0"/>
     </joint>
-    <joint name="chassis-base" type="fixed">
-        <parent link="base"/>
-        <child link="chassis"/>
-        <origin xyz="${chassis_joint_offset} 0 0"/>
-    </joint>
-    <joint name="left_back_wheel-base" type="continuous">
-        <parent link="base"/>
-        <child link="left_back_wheel"/>
-        <origin xyz="${backwheel_offset} ${leftwheel_offset} 0" rpy="${left_roll} 0 0"/>
-        <axis xyz="0 0 1"/>
-    </joint>
-    <joint name="right_back_wheel-base" type="continuous">
-        <parent link="base"/>
-        <child link="right_back_wheel"/>
-        <origin xyz="${backwheel_offset} ${rightwheel_offset} 0" rpy="${right_roll} 0 0"/>
-        <axis xyz="0 0 -1"/>
-    </joint>
-    <joint name="left_front_wheel-base" type="continuous">
-        <parent link="base"/>
-        <child link="left_front_wheel"/>
-        <origin xyz="${frontwheel_offset} ${leftwheel_offset} 0" rpy="${left_roll} 0 0"/>
-        <axis xyz="0 0 1"/>
-    </joint>
-    <joint name="right_front_wheel-base" type="continuous">
-        <parent link="base"/>
-        <child link="right_front_wheel"/>
-        <origin xyz="${frontwheel_offset} ${rightwheel_offset} 0" rpy="${right_roll} 0 0"/>
-        <axis xyz="0 0 -1"/>
-    </joint>
+    <!-- Wheel link-joints -->
+    <xacro:macro name="wheel_link" params="pos_x pos_y">
+        <link name="${pos_x}_${pos_y}_wheel_link">
+            <visual>
+                <geometry>
+                    <mesh filename="package://bot/description/meshes/model-wheel_part_curve.dae" scale="${scale}"/>
+                </geometry>
+                <xacro:scaled_origin_rpy x="0" y="0"  z="0" roll="0" pitch="0" yaw="0"/>
+            </visual>
+            <collision>
+                <geometry>
+                    <mesh filename="package://bot/description/meshes/model-wheel_part_curve.dae" scale="${scale}"/>
+                </geometry>
+                <xacro:scaled_origin_rpy x="0" y="0"  z="0" roll="0" pitch="0" yaw="0"/>
+            </collision>
+            <xacro:inertial_cylinder mass="${wheel_mass}" length="${total_wheel_length}" radius="${actual_wheel_radius}">
+                <!-- <origin xyz="0 0 0" rpy="0 0 0"/> -->
+            <xacro:scaled_origin_rpy x="0" y="0"  z="0" roll="0" pitch="0" yaw="0"/>
+            </xacro:inertial_cylinder>
+        </link>
+    </xacro:macro>
+    <xacro:wheel_link pos_x="left" pos_y="back"/>
+    <xacro:wheel_link pos_x="right" pos_y="back"/>
+    <xacro:wheel_link pos_x="left" pos_y="front"/>
+    <xacro:wheel_link pos_x="right" pos_y="front"/>
+    <xacro:macro name="wheel_joint" params="pos_x pos_y axis">
+        <xacro:if value="${pos_x == 'left'}">
+            <xacro:property name="wheel_x" value="10.0"/>
+            <xacro:property name="wheel_turn" value="${left_roll}"/>
+        </xacro:if>
+        <xacro:if value="${pos_x == 'right'}">
+            <xacro:property name="wheel_x" value="10.0"/>
+            <xacro:property name="wheel_turn" value="${right_roll}"/>
+        </xacro:if>
+        <xacro:if value="${pos_y == 'back'}">
+            <xacro:property name="wheel_y" value="10.0"/>
+        </xacro:if>
+        <xacro:if value="${pos_y == 'front'}">
+            <xacro:property name="wheel_y" value="10.0"/>
+        </xacro:if>
+        <joint name="${pos_x}_${pos_y}_wheel_joint" type="continuous">
+            <parent link="base_link"/>
+            <child link="${pos_x}_${pos_y}_wheel_link"/>
+            <origin xyz="${wheel_x} ${wheel_y} 0" rpy="${wheel_turn} 0 0"/>
+            <xacro:scaled_origin_rpy x="${wheel_x}" y="${wheel_y}"  z="0" roll="${wheel_turn}" pitch="0" yaw="0"/>
+            <axis xyz="0 0 ${axis}"/>
+        </joint>
+    </xacro:macro>
+    <xacro:wheel_joint pos_x="left" pos_y="back" axis="1"/>
+    <xacro:wheel_joint pos_x="right" pos_y="back" axis="-1"/>
+    <xacro:wheel_joint pos_x="left" pos_y="front" axis="1"/>
+    <xacro:wheel_joint pos_x="right" pos_y="front" axis="-1"/>
 </robot>

File: implement_bot/description/base_properties.xacro (robot description, xacro)
@@ -5,28 +5,38 @@
 -->
 <robot xmlns:xacro="http://www.ros.org/wiki/xacro" >
-    <!-- Constant Variables -->
+    <!-- Constants -->
     <xacro:property name="left_roll" value="${-pi/2}"/>
     <xacro:property name="right_roll" value="${pi/2}"/>
-    <!-- Independent Variables -->
-    <xacro:property name="scale" value="1.0"/>
-    <xacro:property name="bot_width" value="0.45"/>
-    <xacro:property name="bot_length" value="0.45"/>
-    <xacro:property name="chassis_height" value="0.15"/>
-    <xacro:property name="chassis_mass" value="0.36"/>
-    <xacro:property name="storage_height" value=""/>
-    <xacro:property name="storage_mass" value="12.0"/>
-    <xacro:property name="top_height" value=""/>
-    <xacro:property name="top_mass" value=""/>
-    <xacro:property name="wheel_radius" value="0.05"/>
-    <xacro:property name="wheel_length" value="0.05"/>
-    <xacro:property name="wheel_mass" value="0.1"/>
-    <!-- Dependent Variables-->
-    <xacro:property name="chassis_joint_offset" value="${-chassis_base/3}"/>
-    <xacro:property name="chassis_link_offset" value="${chassis_base/2}"/>
-    <xacro:property name="chassis_height_offset" value="${chassis_height/2}"/>
-    <xacro:property name="frontwheel_offset" value="${((chassis_base) - (chassis_joint_offset))}"/>
-    <xacro:property name="backwheel_offset" value="${-((chassis_base) - (chassis_joint_offset))}"/>
-    <xacro:property name="leftwheel_offset" value="${(chassis_base/2) + (wheel_length/2)}"/>
-    <xacro:property name="rightwheel_offset" value="${-(chassis_base/2) + (wheel_length/2)}"/>
+    <!-- Variables -->
+    <xacro:property name="scale_val" value="1.0"/>
+    <xacro:property name="scale" value="${scale_val} ${scale_val} ${scale_val}"/>
+    <xacro:property name="bot_pos_x" value="0.0"/>
+    <xacro:property name="bot_pos_y" value="0.0"/>
+    <xacro:property name="bot_pos_z" value="0.0"/>
+    <xacro:property name="actual_bot_width" value="10.0"/>
+    <xacro:property name="actual_bot_length" value="10.0"/>
+    <xacro:property name="actual_chassis_height" value="10.0"/>
+    <xacro:property name="chassis_mass" value="10.0"/>
+    <xacro:property name="actual_storage_height" value="10.0"/>
+    <xacro:property name="storage_mass" value="10.0"/>
+    <xacro:property name="actual_top_height" value="10.0"/>
+    <xacro:property name="top_mass" value="10.0"/>
+    <xacro:property name="actual_wheel_radius" value="10.0"/>
+    <xacro:property name="actual_wheel_thickness" value="10.0"/>
+    <xacro:property name="actual_shaft_length" value="10.0"/>
+    <xacro:property name="total_wheel_length" value="${actual_shaft_length + actual_wheel_thickness}"/>
+    <xacro:property name="wheel_mass" value="10.0"/>
+    <!-- Macros-->
+    <xacro:macro name="scaled_origin" params="x y z">
+        <origin xyz="   ${bot_pos_x + (x * scale_val)}
+                        ${bot_pos_y + (y * scale_val)}
+                        ${bot_pos_z + (z * scale_val)}" />
+    </xacro:macro>
+    <xacro:macro name="scaled_origin_rpy" params="x y z roll pitch yaw">
+        <origin xyz="   ${bot_pos_x + (x * scale_val)}
+                        ${bot_pos_y + (y * scale_val)}
+                        ${bot_pos_z + (z * scale_val)}"
+                rpy="${roll} ${pitch} ${yaw}"/>
+    </xacro:macro>
     <!-- Materials -->
     <material name="white">
@@ -45,7 +55,6 @@
         <color rgba="1 0 0 1"/>
     </material>
-    <!-- Inertial Variables -->
+    <!-- Inertials -->
     <!-- Specify some standard inertial calculations https://en.wikipedia.org/wiki/List_of_moments_of_inertia -->
-    <!-- These make use of xacro's mathematical functionality -->
     <xacro:macro name="inertial_sphere" params="mass radius *origin">
         <inertial>
@@ -61,7 +70,7 @@
             <xacro:insert_block name="origin"/>
             <mass value="${mass}" />
-            <inertia ixx="${(1/12) * mass * (y*y+z*z)}" ixy="0.0" ixz="0.0"
-                    iyy="${(1/12) * mass * (x*x+z*z)}" iyz="0.0"
-                    izz="${(1/12) * mass * (x*x+y*y)}" />
+            <inertia ixx="${(1/12) * (y*y+z*z)}" ixy="0.0" ixz="0.0"
+                    iyy="${(1/12) * (x*x+z*z)}" iyz="0.0"
+                    izz="${(1/12) * (x*x+y*y)}" />
         </inertial>
     </xacro:macro>

File: implement_bot/description/gazebo_control.xacro (robot description, xacro)
@@ -35,5 +35,5 @@
             <!-- Output -->
             <odometry_frame>odom</odometry_frame>
-            <robot_base_frame>base</robot_base_frame>
+            <robot_base_frame>base_link</robot_base_frame>
             <publish_odom>true</publish_odom>
             <publish_odom_tf>true</publish_odom_tf>

File: implement_bot/description/main_urdf.xacro (robot description, xacro)
@@ -1,5 +1,5 @@
 <?xml version="1.0"?>
 <!-- loaded urdf file for robot-->
-<robot xmlns:xacro="http://www.ros.org/wiki/xacro"  name="robot">
+<robot xmlns:xacro="http://www.ros.org/wiki/xacro"  name="robot1">
     <xacro:property name="use_ros2_control" value="true"/>
     <xacro:if value="${use_ros2_control}">
@@ -7,7 +7,7 @@
     </xacro:if>
     <xacro:unless value="${use_ros2_control}">
-        <xacro:include filename="gazebo_control.xacro"/>
+        <!-- <xacro:include filename="gazebo_control.xacro"/> -->
     </xacro:unless>
-    <xacro:include filename="robot_core_actual.xacro"/>
-    <xacro:include filename="lidar.xacro"/>
+    <xacro:include filename="base_actual.xacro"/>
+    <!-- <xacro:include filename="sensors.xacro"/> -->
 </robot>
