Commit message: slight fix of measuremtns & working lidar

File: implement_bot/description/base_actual.xacro (robot description, xacro)
@@ -12,12 +12,12 @@
     </link>
     <joint name="base_joint" type="fixed">
-        <parent link="base_footprint"/>
-        <child link="base_link"/>
-        <origin xyz="0 0 0" rpy="0 0 0"/>
+        <parent link="base_link"/>
+        <child link="base_footprint"/>
+        <origin xyz="0 0 -0.01" rpy="0 0 0"/>
     </joint>
     <!-- <link name="odom">
     </link>
     <joint name="base_odom" type="fixed">
-        <parent link="base_footprint"/>
+        <parent link="base_link"/>
         <child link="odom"/>
         <origin xyz="0 0 0" rpy="0 0 0"/>
@@ -27,5 +27,5 @@
         <visual>
             <geometry>
-                <mesh filename="package://bot/description/meshes/model-chassis_part.dae" scale="${scale}"/>
+                <mesh filename="package://implement_bot/description/meshes/model-chassis_part.dae" scale="${scale}"/>
             </geometry>
             <xacro:scaled_origin x="0.0" y="0.0" z="0.0"/>
@@ -33,10 +33,9 @@
         <collision>
             <geometry>
-                <mesh filename="package://bot/description/meshes/model-chassis_part.dae" scale="${scale}"/>
+                <mesh filename="package://implement_bot/description/meshes/model-chassis_part.dae" scale="${scale}"/>
             </geometry>
             <xacro:scaled_origin x="0.0" y="0.0" z="0.0"/>
         </collision>
         <xacro:inertial_box mass="${chassis_mass}" x="${actual_bot_width}" y="${actual_bot_length}" z="${actual_chassis_height}">
-            <!-- <origin xyz="0 0 0" rpy="0 0 0"/> -->
             <xacro:scaled_origin_rpy x="0" y="0"  z="0" roll="0" pitch="0" yaw="0"/>
         </xacro:inertial_box>
@@ -52,17 +51,16 @@
             <visual>
                 <geometry>
-                    <mesh filename="package://bot/description/meshes/model-wheel_part_curve.dae" scale="${scale}"/>
+                    <mesh filename="package://implement_bot/description/meshes/model-wheel_part_curve.dae" scale="${scale}"/>
                 </geometry>
-                <xacro:scaled_origin_rpy x="0" y="0"  z="0" roll="0" pitch="0" yaw="0"/>
+                <xacro:scaled_origin_rpy x="${-(actual_wheel_thickness/2) - actual_shaft_length}" y="${actual_wheel_radius}"  z="-0.032" roll="0" pitch="0" yaw="0"/>
             </visual>
             <collision>
                 <geometry>
-                    <mesh filename="package://bot/description/meshes/model-wheel_part_curve.dae" scale="${scale}"/>
+                    <mesh filename="package://implement_bot/description/meshes/model-wheel_part_curve.dae" scale="${scale}"/>
                 </geometry>
-                <xacro:scaled_origin_rpy x="0" y="0"  z="0" roll="0" pitch="0" yaw="0"/>
+                <xacro:scaled_origin_rpy x="${-(actual_wheel_thickness/2) - actual_shaft_length}" y="${actual_wheel_radius}"  z="-0.032" roll="0" pitch="0" yaw="0"/>
             </collision>
-            <xacro:inertial_cylinder mass="${wheel_mass}" length="${total_wheel_length}" radius="${actual_wheel_radius}">
-                <!-- <origin xyz="0 0 0" rpy="0 0 0"/> -->
-            <xacro:scaled_origin_rpy x="0" y="0"  z="0" roll="0" pitch="0" yaw="0"/>
+            <xacro:inertial_cylinder mass="${wheel_mass}" length="${actual_wheel_thickness}" radius="${actual_wheel_radius}">
+                <xacro:scaled_origin_rpy x="${-(actual_wheel_thickness/2) - actual_shaft_length}" y="${actual_wheel_radius}"  z="-0.032" roll="0" pitch="0" yaw="0"/>
             </xacro:inertial_cylinder>
         </link>
@@ -74,24 +72,28 @@
     <xacro:macro name="wheel_joint" params="pos_x pos_y axis">
         <xacro:if value="${pos_x == 'left'}">
-            <xacro:property name="wheel_x" value="10.0"/>
-            <xacro:property name="wheel_turn" value="${left_roll}"/>
+            <xacro:property name="wheel_x" value="${-actual_bot_width}"/>
+            <xacro:property name="wheel_turn" value="${pi}"/>
         </xacro:if>
         <xacro:if value="${pos_x == 'right'}">
-            <xacro:property name="wheel_x" value="10.0"/>
-            <xacro:property name="wheel_turn" value="${right_roll}"/>
+            <xacro:property name="wheel_x" value="${actual_bot_width}"/>
+            <xacro:property name="wheel_turn" value="0"/>
         </xacro:if>
         <xacro:if value="${pos_y == 'back'}">
-            <xacro:property name="wheel_y" value="10.0"/>
+            <xacro:property name="wheel_y" value="${-actual_bot_length}"/>
         </xacro:if>
         <xacro:if value="${pos_y == 'front'}">
-            <xacro:property name="wheel_y" value="10.0"/>
+            <xacro:property name="wheel_y" value="${actual_bot_length}"/>
         </xacro:if>
         <joint name="${pos_x}_${pos_y}_wheel_joint" type="continuous">
-            <parent link="base_link"/>
+            <parent link="chassis_link"/>
             <child link="${pos_x}_${pos_y}_wheel_link"/>
-            <origin xyz="${wheel_x} ${wheel_y} 0" rpy="${wheel_turn} 0 0"/>
-            <xacro:scaled_origin_rpy x="${wheel_x}" y="${wheel_y}"  z="0" roll="${wheel_turn}" pitch="0" yaw="0"/>
-            <axis xyz="0 0 ${axis}"/>
+            <xacro:scaled_origin_rpy x="${wheel_x}" y="${wheel_y}"  z="${actual_wheel_radius/2}" roll="0" pitch="${wheel_turn}" yaw="0"/>
+            <axis xyz="${axis} 0 0"/>
         </joint>
+        <!-- <gazebo reference="${pos_x}_${pos_y}_wheel_link">
+            <material>Gazebo/Blue</material>
+            <mu1 value="0.1"/>
+            <mu2 value="0.1"/>
+         </gazebo> -->
     </xacro:macro>
     <xacro:wheel_joint pos_x="left" pos_y="back" axis="1"/>

File: implement_bot/description/base_prac.xacro (robot description, xacro)
@@ -5,5 +5,5 @@
 <robot xmlns:xacro="http://www.ros.org/wiki/xacro">
     <!-- Inertial xacro-->
-    <xacro:include filename="inertial_macros.xacro"/>
+    <xacro:include filename="base_properties.xacro"/>
     <!-- Static Variables -->
     <xacro:property name="left_roll" value="${-pi/2}"/>
@@ -25,5 +25,5 @@
     <xacro:property name="rightwheel_offset" value="-${(chassis_base/2) + (wheel_length/2)}"/>
     <!-- Materials -->
-    <material name="white">
+    <!-- <material name="white">
         <color rgba="1 1 1 1" />
     </material>
@@ -39,5 +39,5 @@
     <material name="red">
         <color rgba="1 0 0 1"/>
-    </material>
+    </material> -->
     <!-- links -->
     <link name="base">

File: implement_bot/description/base_properties.xacro (robot description, xacro)
@@ -13,18 +13,18 @@
     <xacro:property name="bot_pos_x" value="0.0"/>
     <xacro:property name="bot_pos_y" value="0.0"/>
-    <xacro:property name="bot_pos_z" value="0.0"/>
-    <xacro:property name="actual_bot_width" value="10.0"/>
-    <xacro:property name="actual_bot_length" value="10.0"/>
-    <xacro:property name="actual_chassis_height" value="10.0"/>
+    <xacro:property name="bot_pos_z" value="-0.019"/>
+    <xacro:property name="actual_bot_width" value="0.25"/>
+    <xacro:property name="actual_bot_length" value="0.15"/>
+    <xacro:property name="actual_chassis_height" value="0.067"/>
     <xacro:property name="chassis_mass" value="10.0"/>
-    <xacro:property name="actual_storage_height" value="10.0"/>
+    <xacro:property name="actual_storage_height" value="1.0"/>
     <xacro:property name="storage_mass" value="10.0"/>
-    <xacro:property name="actual_top_height" value="10.0"/>
+    <xacro:property name="actual_top_height" value="1.0"/>
     <xacro:property name="top_mass" value="10.0"/>
-    <xacro:property name="actual_wheel_radius" value="10.0"/>
-    <xacro:property name="actual_wheel_thickness" value="10.0"/>
-    <xacro:property name="actual_shaft_length" value="10.0"/>
+    <xacro:property name="actual_wheel_radius" value="0.1275"/>
+    <xacro:property name="actual_wheel_thickness" value="0.1"/>
+    <xacro:property name="actual_shaft_length" value="0.2"/>
     <xacro:property name="total_wheel_length" value="${actual_shaft_length + actual_wheel_thickness}"/>
-    <xacro:property name="wheel_mass" value="10.0"/>
+    <xacro:property name="wheel_mass" value="5.0"/>
     <!-- Macros-->
     <xacro:macro name="scaled_origin" params="x y z">

File: implement_bot/description/gazebo_control.xacro (robot description, xacro)
@@ -26,6 +26,6 @@
         <plugin name="drive" filename="libgazebo_ros_diff_drive.so">
             <!-- Wheel information -->
-            <left_joint>left_back_wheel-base</left_joint>
-            <right_joint>right_back_wheel-base</right_joint>
+            <left_joint>left_back_wheel_joint</left_joint>
+            <right_joint>right_back_wheel_joint</right_joint>
             <wheel_separation>0.35</wheel_separation>
             <wheel_diameter>0.1</wheel_diameter>
@@ -47,8 +47,8 @@
         <plugin name="gazebo_ros_joint_state_publisher" filename="libgazebo_ros_joint_state_publisher.so">
             <update_rate>20</update_rate>
-            <joint_name>left_back_wheel-base</joint_name>
-            <joint_name>right_back_wheel-base</joint_name>
-            <joint_name>left_front_wheel-base</joint_name>
-            <joint_name>right_front_wheel-base</joint_name>
+            <joint_name>left_back_wheel_joint</joint_name>
+            <joint_name>right_back_wheel_joint</joint_name>
+            <joint_name>left_front_wheel_joint</joint_name>
+            <joint_name>right_front_wheel_joint</joint_name>
         </plugin>
     </gazebo>

File: implement_bot/description/main_urdf.xacro (robot description, xacro)
@@ -7,7 +7,7 @@
     </xacro:if>
     <xacro:unless value="${use_ros2_control}">
-        <!-- <xacro:include filename="gazebo_control.xacro"/> -->
+        <xacro:include filename="gazebo_control.xacro"/>
     </xacro:unless>
     <xacro:include filename="base_actual.xacro"/>
-    <!-- <xacro:include filename="sensors.xacro"/> -->
+    <xacro:include filename="sensors.xacro"/>
 </robot>

File: implement_bot/description/ros2_control.xacro (robot description, xacro)
@@ -1,9 +1,10 @@
 <?xml version="1.0"?>
 <robot xmlns:xacro="http://www.ros.org/wiki/xacro">
+    <!-- For Real-life Robot Interface -->
     <ros2_control name="botSys" type="system">
         <hardware>
             <plugin>gazebo_ros2_control/GazeboSystem</plugin>
         </hardware>
-        <joint name="left_back_wheel-base">
+        <joint name='left_back_wheel_joint'>
             <command_interface name="velocity">
                 <param name="min">-10</param>
@@ -13,5 +14,5 @@
             <state_interface name="position"/>
         </joint>
-        <joint name="right_back_wheel-base">
+        <joint name='right_back_wheel_joint'>
             <command_interface name="velocity">
                 <param name="min">-10</param>
@@ -21,5 +22,5 @@
             <state_interface name="position"/>
         </joint>
-        <joint name="left_front_wheel-base">
+        <joint name='left_front_wheel_joint'>
             <command_interface name="velocity">
                 <param name="min">-10</param>
@@ -29,5 +30,5 @@
             <state_interface name="position"/>
         </joint>
-        <joint name="right_front_wheel-base">
+        <joint name='right_front_wheel_joint'>
             <command_interface name="velocity">
                 <param name="min">-10</param>
@@ -38,18 +39,9 @@
         </joint>
     </ros2_control>
+    <!-- For Gazebo Simulation of ROS2 Control -->
     <gazebo>
-        <plugin name="controlPlugin" filename="libgazebo_ros2_control.so">
-            <parameters>$(find implement_bot)/config/my_controllers.yaml</parameters>
+        <plugin name="ros2_controller" filename="libgazebo_ros2_control.so">
+            <parameters>$(find implement_bot)/config/controller_params.yaml</parameters>
         </plugin>
     </gazebo>
-    <!-- <gazebo>
-        <plugin name="gazebo_ros_joint_state_publisher"
-            filename="libgazebo_ros_joint_state_publisher.so">
-            <update_rate>20</update_rate>
-            <joint_name>left_back_wheel-base</joint_name>
-            <joint_name>right_back_wheel-base</joint_name>
-            <joint_name>left_front_wheel-base</joint_name>
-            <joint_name>right_front_wheel-base</joint_name>
-        </plugin>
-    </gazebo> -->
 </robot>

File: implement_bot/description/sensors.xacro (robot description, xacro)
@@ -1,35 +1,40 @@
 <?xml version="1.0"?>
-<robot xmlns.xacro="http://www.ros.org/wiki/xacro">
-    <joint name="laser_joint" type="fixed">
-        <parent link="chassis"/>
-        <child link="laser_frame"/>
-        <origin xyz="0.1 0 0.2" rpy="0 0 0"/>
-    </joint>
-    <link name="laser_frame">
+<robot xmlns:xacro="http://www.ros.org/wiki/xacro">
+    <link name="lidar_link">
         <visual>
             <geometry>
                 <cylinder radius="0.05" length="0.04"/>
             </geometry>
-            <material name="red"/>
+            <origin xyz="0.0 0.0 0.0" rpy="0.0 0.0 ${pi}"/>
+            <material name="black"/>
         </visual>
+        <!-- <xacro:lidar_inertia xyz="0.0 0.0 0.0" rpy="0.0 0.0 0.0"/> -->
         <collision>
             <geometry>
                 <cylinder radius="0.05" length="0.04"/>
             </geometry>
+            <origin xyz="0.0 0.0 0.0" rpy="0.0 0.0 0.0"/>
         </collision>
-        <inertial_cylinder mass="0.1" length="0.04" radius="0.05">
-            <origin xyz="0 0 0" rpy="0 0 0"/>
-        </inertial_cylinder>
     </link>
+    <joint name="lidar_link_joint" type="fixed">
+        <parent link="base_link"/>
+        <child link="lidar_link"/>
+        <origin xyz="0.0 0.0 ${scale_val* 0.2116}" rpy="0.0 0.0 0.0"/>
+    </joint>
+    <link name="laser_frame" />
+    <joint name="lidar_frame_joint" type="fixed">
+        <parent link="lidar_link"/>
+        <child link="laser_frame"/>
+        <origin xyz="0.0 0.0 ${scale_val* 0.025101}" rpy="0.0 0.0 0.0"/>
+    </joint>
     <gazebo reference="laser_frame">
-        <material>Gazebo/Red</material>
         <sensor name="laser" type="ray">
             <pose> 0 0 0 0 0 0 </pose>
             <visualize>true</visualize>
-            <update_rate>50</update_rate>
+            <update_rate>10</update_rate>
             <ray>
                 <scan>
                     <horizontal>
-                        <samples>360</samples>
+                        <samples>720</samples>
                         <min_angle>-3.14</min_angle>
                         <max_angle>3.14</max_angle>
@@ -37,11 +42,11 @@
                 </scan>
                 <range>
-                    <min>0.3</min>
+                    <min>0.1</min>
                     <max>12</max>
                 </range>
             </ray>
-            <plugin name="laser_controller" filename="libgazebo_ros_ray_sensor.so">
+            <plugin name="lidar_gazebo" filename="libgazebo_ros_ray_sensor.so">
                 <ros>
-                    <remapping>~/out:=scan</remapping>
+                    <argument>~/out:=scan</argument>
                 </ros>
                 <output_type>sensor_msgs/LaserScan</output_type>
