Commit message: fixed urdf. still inaccurate. need simpler dae files

File: implement_bot/description/base_actual.xacro (robot description, xacro)
@@ -44,5 +44,5 @@
         <parent link="base_link"/>
         <child link="chassis_link"/>
-        <xacro:scaled_origin x="0.0" y="0.0" z="0.0"/>
+        <xacro:scaled_origin x="${bot_pos_x}" y="${bot_pos_y}" z="${bot_pos_z}"/>
     </joint>
     <!-- Wheel link-joints -->
@@ -53,5 +53,5 @@
                     <mesh filename="package://implement_bot/description/meshes/model-wheel_part_curve.dae" scale="${scale}"/>
                 </geometry>
-                <xacro:scaled_origin_rpy x="${-(actual_wheel_thickness/2) - actual_shaft_length}" y="${actual_wheel_radius}"  z="-0.032" roll="0" pitch="0" yaw="0"/>
+                <xacro:scaled_origin_rpy x="${-actual_shaft_length*2 -(actual_wheel_thickness/2)}" y="${actual_wheel_radius + actual_shaft_thickness}"  z="${-actual_wheel_radius/2 + actual_shaft_thickness*2/3}" roll="0" pitch="0" yaw="0"/>
             </visual>
             <collision>
@@ -59,8 +59,8 @@
                     <mesh filename="package://implement_bot/description/meshes/model-wheel_part_curve.dae" scale="${scale}"/>
                 </geometry>
-                <xacro:scaled_origin_rpy x="${-(actual_wheel_thickness/2) - actual_shaft_length}" y="${actual_wheel_radius}"  z="-0.032" roll="0" pitch="0" yaw="0"/>
+                <xacro:scaled_origin_rpy x="${-actual_shaft_length*2 -(actual_wheel_thickness/2)}" y="${actual_wheel_radius + actual_shaft_thickness}"  z="${-actual_wheel_radius/2 + actual_shaft_thickness*2/3}" roll="0" pitch="0" yaw="0"/>
             </collision>
             <xacro:inertial_cylinder mass="${wheel_mass}" length="${actual_wheel_thickness}" radius="${actual_wheel_radius}">
-                <xacro:scaled_origin_rpy x="${-(actual_wheel_thickness/2) - actual_shaft_length}" y="${actual_wheel_radius}"  z="-0.032" roll="0" pitch="0" yaw="0"/>
+                <xacro:scaled_origin_rpy x="${-actual_shaft_length*2 -(actual_wheel_thickness/2)}" y="${actual_wheel_radius + actual_shaft_thickness}"  z="${-actual_wheel_radius/2 + actual_shaft_thickness*2/3}" roll="0" pitch="0" yaw="0"/>
             </xacro:inertial_cylinder>
         </link>
@@ -72,16 +72,16 @@
     <xacro:macro name="wheel_joint" params="pos_x pos_y axis">
         <xacro:if value="${pos_x == 'left'}">
-            <xacro:property name="wheel_x" value="${-actual_bot_width}"/>
+            <xacro:property name="wheel_x" value="${-(actual_bot_width/2) - actual_wheel_radius}"/>
             <xacro:property name="wheel_turn" value="${pi}"/>
         </xacro:if>
         <xacro:if value="${pos_x == 'right'}">
-            <xacro:property name="wheel_x" value="${actual_bot_width}"/>
+            <xacro:property name="wheel_x" value="${(actual_bot_width/2) + actual_wheel_radius}"/>
             <xacro:property name="wheel_turn" value="0"/>
         </xacro:if>
         <xacro:if value="${pos_y == 'back'}">
-            <xacro:property name="wheel_y" value="${-actual_bot_length}"/>
+            <xacro:property name="wheel_y" value="${-(actual_bot_length/2 - actual_wheel_radius)}"/>
         </xacro:if>
         <xacro:if value="${pos_y == 'front'}">
-            <xacro:property name="wheel_y" value="${actual_bot_length}"/>
+            <xacro:property name="wheel_y" value="${(actual_bot_length/2 - actual_wheel_radius)}"/>
         </xacro:if>
         <joint name="${pos_x}_${pos_y}_wheel_joint" type="continuous">
@@ -91,9 +91,9 @@
             <axis xyz="${axis} 0 0"/>
         </joint>
-        <!-- <gazebo reference="${pos_x}_${pos_y}_wheel_link">
+        <gazebo reference="${pos_x}_${pos_y}_wheel_link">
             <material>Gazebo/Blue</material>
-            <mu1 value="0.1"/>
-            <mu2 value="0.1"/>
-         </gazebo> -->
+            <mu1 value="1.0"/>
+            <mu2 value="0.125"/>
+         </gazebo>
     </xacro:macro>
     <xacro:wheel_joint pos_x="left" pos_y="back" axis="1"/>

File: implement_bot/description/base_properties.xacro (robot description, xacro)
@@ -8,23 +8,26 @@
     <xacro:property name="left_roll" value="${-pi/2}"/>
     <xacro:property name="right_roll" value="${pi/2}"/>
+    <xacro:property name="smol_offset" value="0.01"/>
+    <xacro:property name="kgmm2_to_kgm2" value="1e-6" />
+    <xacro:property name="some_value" value="0.5" />
     <!-- Variables -->
     <xacro:property name="scale_val" value="1.0"/>
     <xacro:property name="scale" value="${scale_val} ${scale_val} ${scale_val}"/>
-    <xacro:property name="bot_pos_x" value="0.0"/>
-    <xacro:property name="bot_pos_y" value="0.0"/>
-    <xacro:property name="bot_pos_z" value="-0.019"/>
-    <xacro:property name="actual_bot_width" value="0.25"/>
-    <xacro:property name="actual_bot_length" value="0.15"/>
-    <xacro:property name="actual_chassis_height" value="0.067"/>
-    <xacro:property name="chassis_mass" value="10.0"/>
-    <xacro:property name="actual_storage_height" value="1.0"/>
+    <xacro:property name="bot_pos_x" value="0.01"/>
+    <xacro:property name="bot_pos_y" value="0.01"/>
+    <xacro:property name="bot_pos_z" value="0.01"/>
+    <xacro:property name="actual_bot_width" value="0.4572"/>
+    <xacro:property name="actual_bot_length" value="0.4572"/>
+    <xacro:property name="actual_chassis_height" value="0.2286"/>
+    <xacro:property name="chassis_mass" value="5.0"/>
+    <xacro:property name="actual_storage_height" value="0.4572"/>
     <xacro:property name="storage_mass" value="10.0"/>
-    <xacro:property name="actual_top_height" value="1.0"/>
+    <xacro:property name="actual_top_height" value="0.1524"/>
     <xacro:property name="top_mass" value="10.0"/>
-    <xacro:property name="actual_wheel_radius" value="0.1275"/>
-    <xacro:property name="actual_wheel_thickness" value="0.1"/>
-    <xacro:property name="actual_shaft_length" value="0.2"/>
-    <xacro:property name="total_wheel_length" value="${actual_shaft_length + actual_wheel_thickness}"/>
-    <xacro:property name="wheel_mass" value="5.0"/>
+    <xacro:property name="actual_wheel_radius" value="${(0.2032)/2}"/>
+    <xacro:property name="actual_wheel_thickness" value="0.0762"/>
+    <xacro:property name="actual_shaft_length" value="0.127"/>
+    <xacro:property name="actual_shaft_thickness" value="0.0232"/>
+    <xacro:property name="wheel_mass" value="2.0"/>
     <!-- Macros-->
     <xacro:macro name="scaled_origin" params="x y z">
@@ -61,6 +64,6 @@
             <xacro:insert_block name="origin"/>
             <mass value="${mass}" />
-            <inertia ixx="${(2/5) * mass * (radius*radius)}" ixy="0.0" ixz="0.0"
-                    iyy="${(2/5) * mass * (radius*radius)}" iyz="0.0"
+            <inertia ixx="${(2/5) * mass * (radius*radius)}" ixy="${mass*some_value}" ixz="${mass*some_value}"
+                    iyy="${(2/5) * mass * (radius*radius)}" iyz="${mass*some_value}"
                     izz="${(2/5) * mass * (radius*radius)}" />
         </inertial>
@@ -70,16 +73,16 @@
             <xacro:insert_block name="origin"/>
             <mass value="${mass}" />
-            <inertia ixx="${(1/12) * (y*y+z*z)}" ixy="0.0" ixz="0.0"
-                    iyy="${(1/12) * (x*x+z*z)}" iyz="0.0"
-                    izz="${(1/12) * (x*x+y*y)}" />
+            <inertia    ixx="${(1/12) * mass * (x*x+z*z)*scale_val}" ixy="${0* some_value}" ixz="${0*some_value}"
+                        iyy="${(1/12) * mass * (y*y+z*z)*scale_val}" iyz="${0*some_value}"
+                        izz="${(1/12) * mass * (y*y+x*x)*scale_val}" />
         </inertial>
     </xacro:macro>
-    <xacro:macro name="inertial_cylinder" params="mass length radius *origin">
+    <xacro:macro name="inertial_cylinder" params="mass length radius *scaled_origin_rpy">
         <inertial>
-            <xacro:insert_block name="origin"/>
+            <xacro:insert_block name="scaled_origin_rpy"/>
             <mass value="${mass}" />
-            <inertia ixx="${(1/12) * mass * (3*radius*radius + length*length)}" ixy="0.0" ixz="0.0"
-                    iyy="${(1/12) * mass * (3*radius*radius + length*length)}" iyz="0.0"
-                    izz="${(1/2) * mass * (radius*radius)}" />
+            <inertia ixx="${(1/12) * mass * (3*radius*radius + length*length) * scale_val}" ixy="${mass*some_value}" ixz="${mass*some_value}"
+                    iyy="${(1/12) * mass * (3*radius*radius + length*length) * scale_val}" iyz="${mass*some_value}"
+                    izz="${(1/2) * mass * (radius*radius) * scale_val}" />
         </inertial>
     </xacro:macro>

File: implement_bot/description/sensors.xacro (robot description, xacro)
@@ -9,5 +9,4 @@
             <material name="black"/>
         </visual>
-        <!-- <xacro:lidar_inertia xyz="0.0 0.0 0.0" rpy="0.0 0.0 0.0"/> -->
         <collision>
             <geometry>
@@ -16,9 +15,12 @@
             <origin xyz="0.0 0.0 0.0" rpy="0.0 0.0 0.0"/>
         </collision>
+        <xacro:inertial_cylinder mass="0.10" length="0.04" radius="0.05">
+                <xacro:scaled_origin_rpy x="0" y="0"  z="0" roll="0" pitch="0" yaw="0"/>
+        </xacro:inertial_cylinder>
     </link>
     <joint name="lidar_link_joint" type="fixed">
-        <parent link="base_link"/>
+        <parent link="chassis_link"/>
         <child link="lidar_link"/>
-        <origin xyz="0.0 0.0 ${scale_val* 0.2116}" rpy="0.0 0.0 0.0"/>
+        <origin xyz="0.0 0.0 ${scale_val* 0.5}" rpy="0.0 0.0 0.0"/>
     </joint>
     <link name="laser_frame" />
@@ -26,5 +28,5 @@
         <parent link="lidar_link"/>
         <child link="laser_frame"/>
-        <origin xyz="0.0 0.0 ${scale_val* 0.025101}" rpy="0.0 0.0 0.0"/>
+        <origin xyz="0.0 0.0 ${scale_val* 0.0}" rpy="0.0 0.0 0.0"/>
     </joint>
     <gazebo reference="laser_frame">

Commit message: urdf fix

File: implement_bot/description/base_actual.xacro (robot description, xacro)
@@ -52,4 +52,5 @@
                 <geometry>
                     <mesh filename="package://implement_bot/description/meshes/model-wheel_part_curve.dae" scale="${scale}"/>
+                    <cylinder radius="${actual_wheel_radius}" length="${actual_wheel_thickness}"/>
                 </geometry>
                 <xacro:scaled_origin_rpy x="${-actual_shaft_length*2 -(actual_wheel_thickness/2)}" y="${actual_wheel_radius + actual_shaft_thickness}"  z="${-actual_wheel_radius/2 + actual_shaft_thickness*2/3}" roll="0" pitch="0" yaw="0"/>
@@ -57,10 +58,13 @@
             <collision>
                 <geometry>
-                    <mesh filename="package://implement_bot/description/meshes/model-wheel_part_curve.dae" scale="${scale}"/>
+                    <!-- <mesh filename="package://implement_bot/description/meshes/model-wheel_part_simple.dae" scale="${scale}"/> -->
+                    <cylinder radius="${actual_wheel_radius}" length="${actual_wheel_thickness}"/>
                 </geometry>
-                <xacro:scaled_origin_rpy x="${-actual_shaft_length*2 -(actual_wheel_thickness/2)}" y="${actual_wheel_radius + actual_shaft_thickness}"  z="${-actual_wheel_radius/2 + actual_shaft_thickness*2/3}" roll="0" pitch="0" yaw="0"/>
+                <origin xyz="0 0 0" rpy="0 ${pi/2} 0 "/>
+                <!-- <xacro:scaled_origin_rpy x="${-actual_shaft_length*2 -(actual_wheel_thickness/2)}" y="${actual_wheel_radius + actual_shaft_thickness}"  z="${-actual_wheel_radius/2 + actual_shaft_thickness*2/3}" roll="0" pitch="0" yaw="0"/> -->
             </collision>
             <xacro:inertial_cylinder mass="${wheel_mass}" length="${actual_wheel_thickness}" radius="${actual_wheel_radius}">
-                <xacro:scaled_origin_rpy x="${-actual_shaft_length*2 -(actual_wheel_thickness/2)}" y="${actual_wheel_radius + actual_shaft_thickness}"  z="${-actual_wheel_radius/2 + actual_shaft_thickness*2/3}" roll="0" pitch="0" yaw="0"/>
+                <origin xyz="0 0 0" rpy="0 ${pi/2} 0 "/>
+                <!-- <xacro:scaled_origin_rpy x="${-actual_shaft_length*2 -(actual_wheel_thickness/2)}" y="${actual_wheel_radius + actual_shaft_thickness}"  z="${-actual_wheel_radius/2 + actual_shaft_thickness*2/3}" roll="0" pitch="0" yaw="0"/> -->
             </xacro:inertial_cylinder>
         </link>
@@ -72,26 +76,28 @@
     <xacro:macro name="wheel_joint" params="pos_x pos_y axis">
         <xacro:if value="${pos_x == 'left'}">
-            <xacro:property name="wheel_x" value="${-(actual_bot_width/2) - actual_wheel_radius}"/>
-            <xacro:property name="wheel_turn" value="${pi}"/>
+            <xacro:property name="wheel_y" value="${+(actual_bot_width/2) + actual_wheel_radius}"/>
+            <xacro:property name="wheel_turn_x" value="0"/>
         </xacro:if>
         <xacro:if value="${pos_x == 'right'}">
-            <xacro:property name="wheel_x" value="${(actual_bot_width/2) + actual_wheel_radius}"/>
-            <xacro:property name="wheel_turn" value="0"/>
+            <xacro:property name="wheel_y" value="${-(actual_bot_width/2) - actual_wheel_radius}"/>
+            <xacro:property name="wheel_turn_x" value="${pi}"/>
         </xacro:if>
         <xacro:if value="${pos_y == 'back'}">
-            <xacro:property name="wheel_y" value="${-(actual_bot_length/2 - actual_wheel_radius)}"/>
+            <xacro:property name="wheel_x" value="${-(actual_bot_length/2 - actual_wheel_radius)}"/>
+            <xacro:property name="wheel_turn_y" value="${pi/2}"/>
         </xacro:if>
         <xacro:if value="${pos_y == 'front'}">
-            <xacro:property name="wheel_y" value="${(actual_bot_length/2 - actual_wheel_radius)}"/>
+            <xacro:property name="wheel_x" value="${(actual_bot_length/2 - actual_wheel_radius)}"/>
+            <xacro:property name="wheel_turn_y" value="${pi/2}"/>
         </xacro:if>
         <joint name="${pos_x}_${pos_y}_wheel_joint" type="continuous">
             <parent link="chassis_link"/>
             <child link="${pos_x}_${pos_y}_wheel_link"/>
-            <xacro:scaled_origin_rpy x="${wheel_x}" y="${wheel_y}"  z="${actual_wheel_radius/2}" roll="0" pitch="${wheel_turn}" yaw="0"/>
+            <xacro:scaled_origin_rpy x="${wheel_x}" y="${wheel_y}"  z="${actual_wheel_radius/2}" roll="0" pitch="${wheel_turn_x}" yaw="${wheel_turn_y}"/>
             <axis xyz="${axis} 0 0"/>
         </joint>
         <gazebo reference="${pos_x}_${pos_y}_wheel_link">
             <material>Gazebo/Blue</material>
-            <mu1 value="1.0"/>
+            <mu1 value="0.250"/>
             <mu2 value="0.125"/>
          </gazebo>

File: implement_bot/description/base_properties.xacro (robot description, xacro)
@@ -6,15 +6,15 @@
 <robot xmlns:xacro="http://www.ros.org/wiki/xacro" >
     <!-- Constants -->
-    <xacro:property name="left_roll" value="${-pi/2}"/>
-    <xacro:property name="right_roll" value="${pi/2}"/>
+    <xacro:property name="right_roll" value="${-pi/2}"/>
+    <xacro:property name="left_roll" value="${pi/2}"/>
     <xacro:property name="smol_offset" value="0.01"/>
     <xacro:property name="kgmm2_to_kgm2" value="1e-6" />
-    <xacro:property name="some_value" value="0.5" />
+    <xacro:property name="some_value" value="0" />
     <!-- Variables -->
     <xacro:property name="scale_val" value="1.0"/>
     <xacro:property name="scale" value="${scale_val} ${scale_val} ${scale_val}"/>
-    <xacro:property name="bot_pos_x" value="0.01"/>
-    <xacro:property name="bot_pos_y" value="0.01"/>
-    <xacro:property name="bot_pos_z" value="0.01"/>
+    <xacro:property name="bot_pos_x" value="0.0"/>
+    <xacro:property name="bot_pos_y" value="0.0"/>
+    <xacro:property name="bot_pos_z" value="${actual_wheel_radius/2 + 0.0}"/>
     <xacro:property name="actual_bot_width" value="0.4572"/>
     <xacro:property name="actual_bot_length" value="0.4572"/>
@@ -32,12 +32,12 @@
     <!-- Macros-->
     <xacro:macro name="scaled_origin" params="x y z">
-        <origin xyz="   ${bot_pos_x + (x * scale_val)}
-                        ${bot_pos_y + (y * scale_val)}
-                        ${bot_pos_z + (z * scale_val)}" />
+        <origin xyz="   ${(x * scale_val)}
+                        ${(y * scale_val)}
+                        ${(z * scale_val)}" />
     </xacro:macro>
     <xacro:macro name="scaled_origin_rpy" params="x y z roll pitch yaw">
-        <origin xyz="   ${bot_pos_x + (x * scale_val)}
-                        ${bot_pos_y + (y * scale_val)}
-                        ${bot_pos_z + (z * scale_val)}"
+        <origin xyz="   ${(x * scale_val)}
+                        ${(y * scale_val)}
+                        ${(z * scale_val)}"
                 rpy="${roll} ${pitch} ${yaw}"/>
     </xacro:macro>

File: implement_bot/description/sensors.xacro (robot description, xacro)
@@ -22,5 +22,5 @@
         <parent link="chassis_link"/>
         <child link="lidar_link"/>
-        <origin xyz="0.0 0.0 ${scale_val* 0.5}" rpy="0.0 0.0 0.0"/>
+        <origin xyz="0.0 0.0 ${(scale_val* (actual_chassis_height + actual_storage_height + actual_top_height)) + 0.02}" rpy="0.0 0.0 0.0"/>
     </joint>
     <link name="laser_frame" />

Commit message: added odom

File: implement_bot/description/base_actual.xacro (robot description, xacro)
@@ -14,13 +14,20 @@
         <parent link="base_link"/>
         <child link="base_footprint"/>
-        <origin xyz="0 0 -0.01" rpy="0 0 0"/>
+        <origin xyz="0 0 0" rpy="0 0 0"/>
     </joint>
-    <!-- <link name="odom">
+    <link name="odom">
     </link>
-    <joint name="base_odom" type="fixed">
-        <parent link="base_link"/>
+    <joint name="odom_base" type="fixed">
+        <parent link="odom"/>
+        <child link="base_link"/>
+        <origin xyz="0 0 0" rpy="0 0 0"/>
+    </joint>
+    <link name="map">
+    </link>
+    <joint name="map_odom" type="fixed">
+        <parent link="map"/>
         <child link="odom"/>
         <origin xyz="0 0 0" rpy="0 0 0"/>
-    </joint> -->
+    </joint>
     <!-- Body link-joints -->
     <link name="chassis_link">

Commit message: added motor joints

File: implement_bot/description/base_actual.xacro (robot description, xacro)
@@ -53,4 +53,41 @@
         <xacro:scaled_origin x="${bot_pos_x}" y="${bot_pos_y}" z="${bot_pos_z}"/>
     </joint>
+    <!-- Motor link-joints -->
+    <xacro:macro name="motor_link_joint" params="pos_x axis">
+        <link name="${pos_x}_motor_link">
+            <visual>
+                <geometry>
+                    <cylinder radius="0.01" length="0.01"/>
+                </geometry>
+                <xacro:scaled_origin_rpy x="${-actual_shaft_length*2 -(actual_wheel_thickness/2)}" y="${actual_wheel_radius + actual_shaft_thickness}"  z="${-actual_wheel_radius/2 + actual_shaft_thickness*2/3}" roll="0" pitch="0" yaw="0"/>
+            </visual>
+            <collision>
+                <geometry>
+                    <cylinder radius="0.01" length="0.01"/>
+                </geometry>
+                <origin xyz="0 0 0" rpy="0 ${pi/2} 0 "/>
+            </collision>
+            <xacro:inertial_cylinder mass="${wheel_mass}" length="${actual_wheel_thickness}" radius="${actual_wheel_radius}">
+                <origin xyz="0 0 0" rpy="0 ${pi/2} 0 "/>
+            </xacro:inertial_cylinder>
+        </link>
+        <xacro:if value="${pos_x == 'left'}">
+            <xacro:property name="wheel_x" value="${+(actual_bot_width/2) + actual_wheel_radius}"/>
+            <xacro:property name="wheel_turn_x" value="0"/>
+        </xacro:if>
+        <xacro:if value="${pos_x == 'right'}">
+            <xacro:property name="wheel_x" value="${-(actual_bot_width/2) - actual_wheel_radius}"/>
+            <xacro:property name="wheel_turn_x" value="${pi}"/>
+        </xacro:if>
+        <xacro:property name="wheel_turn_y" value="${pi/2}"/>
+        <joint name="${pos_x}_motor_joint" type="continuous">
+            <parent link="chassis_link"/>
+            <child link="${pos_x}_motor_link"/>
+            <xacro:scaled_origin_rpy x="0.0" y="${wheel_x}"  z="${actual_wheel_radius/2}" roll="0" pitch="${wheel_turn_x}" yaw="${wheel_turn_y}"/>
+            <axis xyz="${axis} 0 0"/>
+        </joint>
+    </xacro:macro>
+    <xacro:motor_link_joint pos_x="left" axis="1"/>
+    <xacro:motor_link_joint pos_x="right" axis="-1"/>
     <!-- Wheel link-joints -->
     <xacro:macro name="wheel_link" params="pos_x pos_y">
@@ -103,4 +140,5 @@
             <xacro:scaled_origin_rpy x="${wheel_x}" y="${wheel_y}"  z="${actual_wheel_radius/2}" roll="0" pitch="${wheel_turn_x}" yaw="${wheel_turn_y}"/>
             <axis xyz="${axis} 0 0"/>
+            <mimic joint="${pos_x}_motor_joint"/>
         </joint>
         <gazebo reference="${pos_x}_${pos_y}_wheel_link">

File: implement_bot/description/ros2_control.xacro (robot description, xacro)
@@ -1,6 +1,6 @@
 <?xml version="1.0"?>
 <robot xmlns:xacro="http://www.ros.org/wiki/xacro">
-    <!-- For Real-life Robot Interface -->
-    <ros2_control name="botSys" type="system">
+    <!-- For Gazebo Hardware Interface -->
+    <ros2_control name="GazBotSys" type="system">
         <hardware>
             <plugin>gazebo_ros2_control/GazeboSystem</plugin>
@@ -38,9 +38,25 @@
             <state_interface name="position"/>
         </joint>
+        <joint name='left_motor_joint'>
+            <command_interface name="velocity">
+                <param name="min">-10</param>
+                <param name="max">10</param>
+            </command_interface>
+            <state_interface name="velocity"/>
+            <state_interface name="position"/>
+        </joint>
+        <joint name='right_motor_joint'>
+            <command_interface name="velocity">
+                <param name="min">-10</param>
+                <param name="max">10</param>
+            </command_interface>
+            <state_interface name="velocity"/>
+            <state_interface name="position"/>
+        </joint>
     </ros2_control>
     <!-- For Gazebo Simulation of ROS2 Control -->
     <gazebo>
         <plugin name="ros2_controller" filename="libgazebo_ros2_control.so">
-            <parameters>$(find implement_bot)/config/controller_params.yaml</parameters>
+            <parameters>$(find implement_bot)/config/gazebo_controller_params.yaml</parameters>
         </plugin>
     </gazebo>

Commit message: finalizing navigation and localization

File: implement_bot/description/base_actual.xacro (robot description, xacro)
@@ -16,4 +16,5 @@
         <origin xyz="0 0 0" rpy="0 0 0"/>
     </joint>
+    <!-- Final Odom used by EFK Node-->
     <link name="odom">
     </link>
@@ -23,4 +24,12 @@
         <origin xyz="0 0 0" rpy="0 0 0"/>
     </joint>
+    <!-- Odom used by AMCL -->
+    <!-- <link name="odom_unrefined">
+    </link>
+    <joint name="amcl_map" type="fixed">
+        <parent link="odom_unrefined"/>
+        <child link="base_link"/>
+        <origin xyz="0 0 0" rpy="0 0 0"/>
+    </joint> -->
     <link name="map">
     </link>
