Commit message: sad

File: implement_bot/description/base_actual.xacro (robot description, xacro)
@@ -91,5 +91,5 @@
         <xacro:property name="wheel_turn_y" value="${pi/2}"/>
         <joint name="${pos_x}_motor_joint" type="fixed">
-            <parent link="chassis_link"/>
+            <parent link="base_link"/>
             <child link="${pos_x}_caster_link"/>
             <xacro:scaled_origin_rpy x="${-(actual_bot_length/2 - actual_wheel_radius*2)}" y="${wheel_x}"  z="0" roll="0" pitch="${wheel_turn_x}" yaw="${wheel_turn_y}"/>

File: implement_bot/description/sensors.xacro (robot description, xacro)
@@ -22,5 +22,5 @@
     <!-- Lidar Joint to Base Link -->
     <joint name="lidar_link_joint" type="fixed">
-        <parent link="chassis_link"/>
+        <parent link="base_link"/>
         <child link="ldlidar_link"/>
         <origin xyz="0.0 0.0 ${(scale_val* (actual_chassis_height + actual_storage_height + actual_top_height)) + 0.02 -0.7}" rpy="0.0 0.0 0.0"/>
@@ -53,5 +53,5 @@
         </xacro:if>
         <joint name="${pos_x}_range_joint" type="fixed">
-            <parent link="chassis_link"/>
+            <parent link="base_link"/>
             <child link="${pos_x}_range_link"/>
             <xacro:scaled_origin_rpy x="${(actual_bot_length/2) + smol_offset}" y="${offset_x + 0.02}"  z="${actual_wheel_radius}" roll="0" pitch="0" yaw="0"/>
@@ -60,7 +60,7 @@
     </xacro:macro>
     <!-- left IR sensor -->
-    <!-- <xacro:range_link_joint pos_x="left"/> -->
+    <xacro:range_link_joint pos_x="left"/>
     <!-- right IR sensor -->
-    <!-- <xacro:range_link_joint pos_x="right"/> -->
+    <xacro:range_link_joint pos_x="right"/>
     <!-- IMU Link -->
     <link name="imu_link">
@@ -83,5 +83,5 @@
     <!-- IMU joint to base link -->
     <joint name="imu_link_joint" type="fixed">
-        <parent link="chassis_link"/>
+        <parent link="base_link"/>
         <child link="imu_link"/>
         <origin xyz="0.0 0.0 ${scale_val* 0.0}" rpy="0.0 0.0 0.0"/>

Commit message: gui updates

File: implement_bot/description/base_actual.xacro (robot description, xacro)
@@ -14,5 +14,5 @@
         <parent link="base_link"/>
         <child link="base_footprint"/>
-        <origin xyz="0 0 0" rpy="0 0 0"/>
+        <origin xyz="0 0 -0.001" rpy="0 0 0"/>
     </joint>
     <!-- Final Odom used by EFK Node-->
@@ -24,12 +24,4 @@
         <origin xyz="0 0 0" rpy="0 0 0"/>
     </joint>
-    <!-- Odom used by AMCL -->
-    <!-- <link name="odom_unrefined">
-    </link>
-    <joint name="amcl_map" type="fixed">
-        <parent link="odom_unrefined"/>
-        <child link="base_link"/>
-        <origin xyz="0 0 0" rpy="0 0 0"/>
-    </joint> -->
     <link name="map">
     </link>
@@ -90,5 +82,5 @@
         </xacro:if>
         <xacro:property name="wheel_turn_y" value="${pi/2}"/>
-        <joint name="${pos_x}_motor_joint" type="fixed">
+        <joint name="${pos_x}_caster_joint" type="fixed">
             <parent link="base_link"/>
             <child link="${pos_x}_caster_link"/>
@@ -148,5 +140,5 @@
         </xacro:if>
         <joint name="${pos_x}_${pos_y}_wheel_joint" type="continuous">
-            <parent link="chassis_link"/>
+            <parent link="base_link"/>
             <child link="${pos_x}_${pos_y}_wheel_link"/>
             <xacro:scaled_origin_rpy x="${wheel_x}" y="${wheel_y}"  z="${actual_wheel_radius/2}" roll="0" pitch="${wheel_turn_x}" yaw="${wheel_turn_y}"/>

File: implement_bot/description/ros2_control.xacro (robot description, xacro)
@@ -13,5 +13,5 @@
             <param name="timeout_ms">0</param>
             <param name="enc_counts_per_rev">60</param>
-            <param name="pid_p">20</param>
+            <param name="pid_p">50</param>
             <param name="pid_d">10</param>
             <param name="pid_i">10</param>

Commit message: some fixes

File: implement_bot/description/base_actual.xacro (robot description, xacro)
@@ -54,4 +54,48 @@
         <xacro:scaled_origin x="${bot_pos_x}" y="${bot_pos_y}" z="${bot_pos_z}"/>
     </joint>
+    <link name="load_link">
+        <visual>
+            <geometry>
+                <mesh filename="package://implement_bot/description/meshes/model-load_part.dae" scale="${scale}"/>
+            </geometry>
+            <xacro:scaled_origin x="0.0" y="0.0" z="0.0"/>
+        </visual>
+        <collision>
+            <geometry>
+                <mesh filename="package://implement_bot/description/meshes/model-load_part.dae" scale="${scale}"/>
+            </geometry>
+            <xacro:scaled_origin x="0.0" y="0.0" z="0.0"/>
+        </collision>
+        <xacro:inertial_box mass="${storage_mass}" x="${actual_bot_width}" y="${actual_bot_length}" z="${actual_storage_height}">
+            <xacro:scaled_origin_rpy x="0" y="0"  z="0" roll="0" pitch="0" yaw="0"/>
+        </xacro:inertial_box>
+    </link>
+    <joint name="load_joint" type="fixed">
+        <parent link="base_link"/>
+        <child link="load_link"/>
+        <xacro:scaled_origin x="${bot_pos_x}" y="${bot_pos_y}" z="${bot_pos_z}"/>
+    </joint>
+    <link name="top_link">
+        <visual>
+            <geometry>
+                <mesh filename="package://implement_bot/description/meshes/model-top_part.dae" scale="${scale}"/>
+            </geometry>
+            <xacro:scaled_origin x="0.0" y="0.0" z="0.0"/>
+        </visual>
+        <collision>
+            <geometry>
+                <mesh filename="package://implement_bot/description/meshes/model-top_part.dae" scale="${scale}"/>
+            </geometry>
+            <xacro:scaled_origin x="0.0" y="0.0" z="0.0"/>
+        </collision>
+        <xacro:inertial_box mass="${top_mass}" x="${actual_bot_width}" y="${actual_bot_length}" z="${actual_top_height}">
+            <xacro:scaled_origin_rpy x="0" y="0"  z="0" roll="0" pitch="0" yaw="0"/>
+        </xacro:inertial_box>
+    </link>
+    <joint name="top_joint" type="fixed">
+        <parent link="base_link"/>
+        <child link="top_link"/>
+        <xacro:scaled_origin x="${bot_pos_x}" y="${bot_pos_y}" z="${bot_pos_z}"/>
+    </joint>
     <!-- Caster link-joints -->
     <xacro:macro name="caster_link_joint" params="pos_x axis">
@@ -85,5 +129,5 @@
             <parent link="base_link"/>
             <child link="${pos_x}_caster_link"/>
-            <xacro:scaled_origin_rpy x="${-(actual_bot_length/2 - actual_wheel_radius*2)}" y="${wheel_x}"  z="0" roll="0" pitch="${wheel_turn_x}" yaw="${wheel_turn_y}"/>
+            <xacro:scaled_origin_rpy x="${-(actual_bot_length/2 - actual_wheel_radius*2)}" y="${wheel_x}"  z="${bot_pos_z}" roll="0" pitch="${wheel_turn_x}" yaw="${wheel_turn_y}"/>
             <axis xyz="${axis} 0 0"/>
         </joint>
@@ -142,5 +186,5 @@
             <parent link="base_link"/>
             <child link="${pos_x}_${pos_y}_wheel_link"/>
-            <xacro:scaled_origin_rpy x="${wheel_x}" y="${wheel_y}"  z="${actual_wheel_radius/2}" roll="0" pitch="${wheel_turn_x}" yaw="${wheel_turn_y}"/>
+            <xacro:scaled_origin_rpy x="${wheel_x}" y="${wheel_y}"  z="${bot_pos_z + (actual_wheel_radius/2)}" roll="0" pitch="${wheel_turn_x}" yaw="${wheel_turn_y}"/>
             <axis xyz="${axis} 0 0"/>
             <mimic joint="${pos_x}_motor_joint"/>

File: implement_bot/description/sensors.xacro (robot description, xacro)
@@ -24,5 +24,5 @@
         <parent link="base_link"/>
         <child link="ldlidar_link"/>
-        <origin xyz="0.0 0.0 ${(scale_val* (actual_chassis_height + actual_storage_height + actual_top_height)) + 0.02 -0.7}" rpy="0.0 0.0 0.0"/>
+        <origin xyz="0.0 0.0 ${(scale_val* (actual_chassis_height + actual_storage_height + actual_top_height + 0.04))}" rpy="0.0 0.0 0.0"/>
         <!-- <origin xyz="0.0 0.0 ${(scale_val* (actual_chassis_height) + 0.02)}" rpy="0.0 0.0 0.0"/> -->
     </joint>
@@ -55,5 +55,5 @@
             <parent link="base_link"/>
             <child link="${pos_x}_range_link"/>
-            <xacro:scaled_origin_rpy x="${(actual_bot_length/2) + smol_offset}" y="${offset_x + 0.02}"  z="${actual_wheel_radius}" roll="0" pitch="0" yaw="0"/>
+            <xacro:scaled_origin_rpy x="${(actual_bot_length/2) + smol_offset}" y="${offset_x + 0.1}"  z="${actual_wheel_radius}" roll="0" pitch="0" yaw="0"/>
             <axis xyz="0 0 0"/>
         </joint>
