Commit message: simple cleaned files

File: implement_bot/description/ros2_control.xacro (robot description, xacro)
@@ -18,14 +18,4 @@
             <param name="pid_o">50</param>
         </hardware>
-        <!-- <joint name='left_front_wheel_joint'>
-            <command_interface name="velocity"/>
-            <state_interface name="velocity"/>
-            <state_interface name="position"/>
-        </joint>
-        <joint name='right_front_wheel_joint'>
-            <command_interface name="velocity"/>
-            <state_interface name="velocity"/>
-            <state_interface name="position"/>
-        </joint> -->
     </ros2_control>
 </robot>

Commit message: adding sensors

File: implement_bot/description/ros2_control.xacro (robot description, xacro)
@@ -18,4 +18,14 @@
             <param name="pid_o">50</param>
         </hardware>
+         <joint name='left_front_wheel_joint'>
+            <command_interface name="velocity"/>
+            <state_interface name="velocity"/>
+            <state_interface name="position"/>
+        </joint>
+        <joint name='right_front_wheel_joint'>
+            <command_interface name="velocity"/>
+            <state_interface name="velocity"/>
+            <state_interface name="position"/>
+        </joint>
     </ros2_control>
 </robot>

File: implement_bot/description/sensors.xacro (robot description, xacro)
@@ -27,5 +27,5 @@
         <!-- <origin xyz="0.0 0.0 ${(scale_val* (actual_chassis_height) + 0.02)}" rpy="0.0 0.0 0.0"/> -->
     </joint>
-    <!-- Macro for Ultrasonic Sensors -->
+    <!-- Macro for IR Sensors -->
     <xacro:macro name="range_link_joint" params="pos_x">
         <link name="${pos_x}_range_link">
@@ -59,7 +59,7 @@
         </joint>
     </xacro:macro>
-    <!-- left ultrasonic sensor -->
+    <!-- left IR sensor -->
     <xacro:range_link_joint pos_x="left"/>
-    <!-- right ultrasonic sensor -->
+    <!-- right IR sensor -->
     <xacro:range_link_joint pos_x="right"/>
     <!-- IMU Link -->

Commit message: bot configure edits

File: implement_bot/description/ros2_control.xacro (robot description, xacro)
@@ -8,6 +8,6 @@
             <param name="right_wheel_name">right_front_wheel_joint</param>
             <param name="loop_rate">30</param>
-            <!-- <param name="device">/dev/serial/by-path/platform-fd500000.pcie-pci-0000:01:00.0-usb-0:1.3:1.0-port0</param> -->
-            <param name="device">/dev/ttyUSB0</param>
+            <param name="device">/dev/serial/by-path/platform-fd500000.pcie-pci-0000:01:00.0-usb-0:1.2:1.0-port0</param>
+            <!-- <param name="device">/dev/serial1</param> -->
             <param name="baud_rate">57600</param>
             <param name="timeout_ms">1000</param>

File: implement_bot/description/sensors.xacro (robot description, xacro)
@@ -24,5 +24,5 @@
         <parent link="chassis_link"/>
         <child link="ldlidar_link"/>
-        <origin xyz="0.0 0.0 ${(scale_val* (actual_chassis_height + actual_storage_height + actual_top_height)) + 0.02}" rpy="0.0 0.0 0.0"/>
+        <origin xyz="0.0 0.0 ${(scale_val* (actual_chassis_height + actual_storage_height + actual_top_height)) + 0.02 -0.7}" rpy="0.0 0.0 0.0"/>
         <!-- <origin xyz="0.0 0.0 ${(scale_val* (actual_chassis_height) + 0.02)}" rpy="0.0 0.0 0.0"/> -->
     </joint>

Commit message: news

File: implement_bot/description/ros2_control.xacro (robot description, xacro)
@@ -17,6 +17,7 @@
             <param name="pid_i">0</param>
             <param name="pid_o">1</param>
-            <param name="left_range_name">left_range</param>
-            <param name="right_range_name">right_range</param>
+            <!-- <param name="left_range_name">left_range</param>
+            <param name="right_range_name">right_range</param> -->
+            <param name="range_name">range</param>
             <param name="imu_name">imu</param>
         </hardware>

File: implement_bot/description/sensors.xacro (robot description, xacro)
@@ -60,7 +60,30 @@
     </xacro:macro>
     <!-- left IR sensor -->
-    <xacro:range_link_joint pos_x="left"/>
+    <!-- <xacro:range_link_joint pos_x="left"/> -->
     <!-- right IR sensor -->
-    <xacro:range_link_joint pos_x="right"/>
+    <!-- <xacro:range_link_joint pos_x="right"/> -->
+    <link name="range_link">
+        <visual>
+            <geometry>
+                <box size="0.015 0.03 0.001"/>
+            </geometry>
+            <xacro:scaled_origin_rpy x="0.0" y="0.0"  z="0.0" roll="0" pitch="0" yaw="0"/>
+        </visual>
+        <collision>
+            <geometry>
+                <box size="0.015 0.03 0.01"/>
+            </geometry>
+            <xacro:scaled_origin_rpy x="0.0" y="0.0"  z="0.0" roll="0" pitch="0" yaw="0"/>
+        </collision>
+        <xacro:inertial_box mass="0.001" x="0.0" y="0.0" z="0.0">
+        <origin xyz="0.0 0 0.0" rpy="-1 0 0"/>
+        </xacro:inertial_box>
+    </link>
+    <joint name="range_joint" type="fixed">
+        <parent link="base_link"/>
+        <child link="range_link"/>
+        <xacro:scaled_origin_rpy x="${(actual_bot_length/2) + smol_offset}" y="0.0"  z="${actual_wheel_radius}" roll="0" pitch="0" yaw="0"/>
+        <axis xyz="0 0 0"/>
+    </joint>
     <!-- IMU Link -->
     <link name="imu_link">
